File: Kicad/stm32F746 GRBL/Power.kicad_sch (KiCad schematic)
At the start: 1 part, among them J13 Screw_Terminal_01x04

Commit message: kicad wip
Parts:
- added C5: 2.2uF, Capacitor_SMD:C_0805_2012Metric_Pad1.18x1.45mm_HandSolder, symbol Device:C_Polarized
- added C6: 0.1uF, Capacitor_SMD:C_0805_2012Metric, symbol Device:C
- added C7, C8: 22uF, Capacitor_SMD:C_0805_2012Metric_Pad1.18x1.45mm_HandSolder, symbol Device:C_Polarized
- added C9: 10uF, Capacitor_Tantalum_SMD:CP_EIA-3528-15_AVX-H_Pad1.50x2.35mm_HandSolder, symbol Device:C_Polarized
- added F1: Polyfuse, Fuse:Fuse_1812_4532Metric_Pad1.30x3.40mm_HandSolder, symbol Device:Polyfuse
- added L1: 6.8uH, Inductor_SMD:L_Bourns_SRP5030T, symbol Device:L
- added R14: 100K, Resistor_SMD:R_0805_2012Metric_Pad1.20x1.40mm_HandSolder, symbol Device:R
- added R15: 13.7K, Resistor_SMD:R_0805_2012Metric_Pad1.20x1.40mm_HandSolder, symbol Device:R
- added U10: LMR51430, Package_TO_SOT_SMD:SOT-23-6, symbol Regulator_Switching:LMR51430
- added U11: LM1117MP-3.3, Package_TO_SOT_SMD:SOT-223-3_TabPin2, symbol Regulator_Linear:LM1117MP-3.3
- J13: value Screw_Terminal_01x04 -> Power Input
Connections:
- net GND: now also J13.3 (Pin_3), C5.2, C7.2, C8.2, C9.2, R15.2, U10.1 (GND), U11.1 (GND)
- net Vdrive: now also J13.2 (Pin_2), F1.1
- new net: C6.2, L1.1, U10.2 (SW)
- new net: C6.1, U10.6 (CB)
- new net: R14.2, R15.1, U10.4 (FB)
- new net: C5.1, F1.2, U10.3 (VIN), U10.5 (EN)
- new net +3.3VP: C9.1, U11.2 (VO)
- new net +5VP: C8.1, L1.2, R14.1, U11.3 (VI)
Other:
- moved on the sheet: J13

Commit message: wip kicad
Connections:
- net Vdrive: now also C5.1, F1.2, U10.3 (VIN), U10.5 (EN); no longer F1.1, J13.1 (Pin_1), J13.2 (Pin_2)
- new net: F1.1, J13.1 (Pin_1), J13.2 (Pin_2)
Other:
- moved on the sheet: J13
Changed lines of the file:
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@@
   (junction (at 165.735 68.58) (diameter 0) (color 0 0 0 0)
   )
-  (junction (at 57.785 52.705) (diameter 0) (color 0 0 0 0)
-  )
-  (junction (at 57.785 60.325) (diameter 0) (color 0 0 0 0)
+  (junction (at 74.295 54.61) (diameter 0) (color 0 0 0 0)
+  )
+  (junction (at 74.295 62.23) (diameter 0) (color 0 0 0 0)
   )
   (junction (at 121.92 54.61) (diameter 0) (color 0 0 0 0)
@@
     (stroke (width 0) (type default))
   )
-  (wire (pts (xy 57.785 57.785) (xy 57.785 60.325))
-    (stroke (width 0) (type default))
-  )
-  (wire (pts (xy 57.785 52.705) (xy 59.69 52.705))
+  (wire (pts (xy 74.295 59.69) (xy 74.295 62.23))
+    (stroke (width 0) (type default))
+  )
+  (wire (pts (xy 74.295 54.61) (xy 72.39 54.61))
     (stroke (width 0) (type default))
   )
@@
     (stroke (width 0) (type default))
   )
-  (wire (pts (xy 57.785 55.245) (xy 57.785 52.705))
+  (wire (pts (xy 74.295 57.15) (xy 74.295 54.61))
     (stroke (width 0) (type default))
   )
@@
     (stroke (width 0) (type default))
   )
-  (wire (pts (xy 53.34 51.435) (xy 53.34 52.705))
-    (stroke (width 0) (type default))
-  )
   (wire (pts (xy 116.205 67.31) (xy 116.205 64.135))
     (stroke (width 0) (type default))
@@
     (stroke (width 0) (type default))
   )
-  (wire (pts (xy 59.69 55.245) (xy 57.785 55.245))
-    (stroke (width 0) (type default))
-  )
-  (wire (pts (xy 53.34 52.705) (xy 57.785 52.705))
+  (wire (pts (xy 72.39 57.15) (xy 74.295 57.15))
+    (stroke (width 0) (type default))
+  )
+  (wire (pts (xy 74.295 54.61) (xy 97.79 54.61))
     (stroke (width 0) (type default))
   )
@@
     (stroke (width 0) (type default))
   )
+  (wire (pts (xy 116.205 48.26) (xy 116.205 54.61))
+    (stroke (width 0) (type default))
+  )
   (wire (pts (xy 165.735 68.58) (xy 165.735 69.85))
     (stroke (width 0) (type default))
@@
     (stroke (width 0) (type default))
   )
-  (wire (pts (xy 57.785 62.23) (xy 57.785 60.325))
+  (wire (pts (xy 74.295 64.135) (xy 74.295 62.23))
     (stroke (width 0) (type default))
   )
@@
     (stroke (width 0) (type default))
   )
-  (wire (pts (xy 88.265 54.61) (xy 88.265 48.895))
-    (stroke (width 0) (type default))
-  )
-  (wire (pts (xy 59.69 57.785) (xy 57.785 57.785))
+  (wire (pts (xy 72.39 59.69) (xy 74.295 59.69))
     (stroke (width 0) (type default))
   )
@@
     (stroke (width 0) (type default))
   )
-  (wire (pts (xy 57.785 60.325) (xy 59.69 60.325))
+  (wire (pts (xy 74.295 62.23) (xy 72.39 62.23))
     (stroke (width 0) (type default))
   )
   (wire (pts (xy 144.145 52.07) (xy 145.415 52.07))
-    (stroke (width 0) (type default))
-  )
-  (wire (pts (xy 88.265 54.61) (xy 97.79 54.61))
     (stroke (width 0) (type default))
   )
@@
     )
   )
+  (symbol (lib_id "power:Vdrive") (at 116.205 48.26 0) (unit 1)
+    (in_bom yes) (on_board yes) (dnp no)
+    (property "Reference" "#PWR097" (at 111.125 52.07 0)
+      (effects (font (size 1.27 1.27)) hide)
+    )
+    (property "Value" "Vdrive" (at 121.285 45.72 0)
+      (effects (font (size 1.27 1.27)))
+    )
+    (property "Footprint" "" (at 116.205 48.26 0)
+      (effects (font (size 1.27 1.27)) hide)
+    )
+    (property "Datasheet" "" (at 116.205 48.26 0)
+      (effects (font (size 1.27 1.27)) hide)
+    )
+    (pin "1")
+    (instances
+      (project "stm32F746 GRBL"
+        (path "/2c79a78e-687a-4954-b7b9-175bc3470bd7/cfe63f02-1987-4919-8e32-0515eff710ca"
+          (reference "#PWR097") (unit 1)
+        )
+      )
+    )
+  )
   (symbol (lib_id "power:GND") (at 226.695 64.77 0) (unit 1)
     (in_bom yes) (on_board yes) (dnp no) (fields_autoplaced)
@@
         (path "/2c79a78e-687a-4954-b7b9-175bc3470bd7/cfe63f02-1987-4919-8e32-0515eff710ca"
           (reference "C6") (unit 1)
-        )
-      )
-    )
-  )
-  (symbol (lib_id "power:Vdrive") (at 53.34 51.435 0) (unit 1)
-    (in_bom yes) (on_board yes) (dnp no)
-    (property "Reference" "#PWR011" (at 48.26 55.245 0)
-      (effects (font (size 1.27 1.27)) hide)
-    )
-    (property "Value" "Vdrive" (at 58.42 48.895 0)
-      (effects (font (size 1.27 1.27)))
-    )
-    (property "Footprint" "" (at 53.34 51.435 0)
-      (effects (font (size 1.27 1.27)) hide)
-    )
-    (property "Datasheet" "" (at 53.34 51.435 0)
-      (effects (font (size 1.27 1.27)) hide)
-    )
-    (pin "1")
-    (instances
-      (project "stm32F746 GRBL"
-        (path "/2c79a78e-687a-4954-b7b9-175bc3470bd7/cfe63f02-1987-4919-8e32-0515eff710ca"
-          (reference "#PWR011") (unit 1)
         )
       )
@@
     )
   )
-  (symbol (lib_id "power:Vdrive") (at 88.265 48.895 0) (unit 1)
-    (in_bom yes) (on_board yes) (dnp no)
-    (property "Reference" "#PWR0138" (at 83.185 52.705 0)
-      (effects (font (size 1.27 1.27)) hide)
-    )
-    (property "Value" "Vdrive" (at 93.345 46.355 0)
-      (effects (font (size 1.27 1.27)))
-    )
-    (property "Footprint" "" (at 88.265 48.895 0)
-      (effects (font (size 1.27 1.27)) hide)
-    )
-    (property "Datasheet" "" (at 88.265 48.895 0)
-      (effects (font (size 1.27 1.27)) hide)
-    )
-    (pin "1")
-    (instances
-      (project "stm32F746 GRBL"
-        (path "/2c79a78e-687a-4954-b7b9-175bc3470bd7/cfe63f02-1987-4919-8e32-0515eff710ca"
-          (reference "#PWR0138") (unit 1)
-        )
-      )
-    )
-  )
   (symbol (lib_id "Device:R") (at 165.735 73.66 0) (mirror y) (unit 1)
     (in_bom yes) (on_board yes) (dnp no)
@@
     )
   )
-  (symbol (lib_id "Connector:Screw_Terminal_01x04") (at 64.77 55.245 0) (unit 1)
-    (in_bom yes) (on_board yes) (dnp no) (fields_autoplaced)
-    (property "Reference" "J13" (at 67.31 55.245 0)
+  (symbol (lib_id "Connector:Screw_Terminal_01x04") (at 67.31 57.15 0) (mirror y) (unit 1)
+    (in_bom yes) (on_board yes) (dnp no) (fields_autoplaced)
+    (property "Reference" "J13" (at 64.77 57.15 0)
       (effects (font (size 1.27 1.27)) (justify left))
     )
-    (property "Value" "Power Input" (at 67.31 57.785 0)
+    (property "Value" "Power Input" (at 64.77 59.69 0)
       (effects (font (size 1.27 1.27)) (justify left))
     )
-    (property "Footprint" "Connector_Phoenix_MSTB:PhoenixContact_MSTBA_2,5_4-G-5,08_1x04_P5.08mm_Horizontal" (at 64.77 55.245 0)
-      (effects (font (size 1.27 1.27)) hide)
-    )
-    (property "Datasheet" "~" (at 64.77 55.245 0)
+    (property "Footprint" "Connector_Phoenix_MSTB:PhoenixContact_MSTBA_2,5_4-G-5,08_1x04_P5.08mm_Horizontal" (at 67.31 57.15 0)
+      (effects (font (size 1.27 1.27)) hide)
+    )
+    (property "Datasheet" "~" (at 67.31 57.15 0)
       (effects (font (size 1.27 1.27)) hide)
     )
@@
     )
   )
-  (symbol (lib_id "power:GND") (at 57.785 62.23 0) (unit 1)
-    (in_bom yes) (on_board yes) (dnp no) (fields_autoplaced)
-    (property "Reference" "#PWR0140" (at 57.785 68.58 0)
-      (effects (font (size 1.27 1.27)) hide)
-    )
-    (property "Value" "GND" (at 57.785 66.04 90)
+  (symbol (lib_id "power:GND") (at 74.295 64.135 0) (mirror y) (unit 1)
+    (in_bom yes) (on_board yes) (dnp no) (fields_autoplaced)
+    (property "Reference" "#PWR0140" (at 74.295 70.485 0)
+      (effects (font (size 1.27 1.27)) hide)
+    )
+    (property "Value" "GND" (at 74.295 67.945 90)
       (effects (font (size 1.27 1.27)) (justify right) hide)
     )
-    (property "Footprint" "" (at 57.785 62.23 0)
-      (effects (font (size 1.27 1.27)) hide)
-    )
-    (property "Datasheet" "" (at 57.785 62.23 0)
-      (effects (font (size 1.27 1.27)) hide)
-    )
+    (property "Footprint" "" (at 74.295 64.135 0)
+      (effects (font (size 1.27 1.27)) hide)
+    )
+    (property "Datasheet" "" (at 74.295 64.135 0)
+      (effects (font (size 1.27 1.27)) hide)
+    )
