File: Kicad/stm32F746 GRBL/Power.kicad_sch (KiCad schematic)
At the start: 12 parts, among them J13 Power Input, U10 LMR51430, U11 LM1117MP-3.3

Commit message: wip kicad
Parts:
- removed F1: Polyfuse, Fuse:Fuse_1812_4532Metric_Pad1.30x3.40mm_HandSolder, symbol Device:Polyfuse
- added F1: Fuse, symbol Device:Fuse
Connections:
- net Vdrive: now also F1.2
- net at J13.1 (Pin_1), J13.2 (Pin_2): now also F1.1
Changed lines of the file:
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@@
+    )
+  )
+  (symbol (lib_id "Device:Fuse") (at 101.6 54.61 90) (unit 1)
+    (in_bom yes) (on_board yes) (dnp no) (fields_autoplaced)
+    (property "Reference" "F1" (at 101.6 49.53 90)
+      (effects (font (size 1.27 1.27)))
+    )
+    (property "Value" "Fuse" (at 101.6 52.07 90)
+      (effects (font (size 1.27 1.27)))
+    )
+    (property "Footprint" "" (at 101.6 56.388 90)
+      (effects (font (size 1.27 1.27)) hide)
+    )
+    (property "Datasheet" "~" (at 101.6 54.61 0)
+      (effects (font (size 1.27 1.27)) hide)
+    )
+    (pin "1")
+    (pin "2")
+    (instances
+      (project "stm32F746 GRBL"
+        (path "/2c79a78e-687a-4954-b7b9-175bc3470bd7/cfe63f02-1987-4919-8e32-0515eff710ca"
+          (reference "F1") (unit 1)
+        )
+      )
     )
   )
@@
         )
       )
-    )
-  )
-  (symbol (lib_id "Device:Polyfuse") (at 101.6 54.61 90) (unit 1)
-    (in_bom yes) (on_board yes) (dnp no) (fields_autoplaced)
-    (property "Reference" "F1" (at 101.6 48.26 90)
-      (effects (font (size 1.27 1.27)))
-    )
-    (property "Value" "Polyfuse" (at 101.6 50.8 90)
-      (effects (font (size 1.27 1.27)))
-    )
-    (property "Footprint" "Fuse:Fuse_1812_4532Metric_Pad1.30x3.40mm_HandSolder" (at 106.68 53.34 0)
-      (effects (font (size 1.27 1.27)) (justify left) hide)
-    )
-    (property "Datasheet" "~" (at 101.6 54.61 0)
-      (effects (font (size 1.27 1.27)) hide)
-    )
-    (pin "1")
-    (pin "2")
-    (instances
-      (project "stm32F746 GRBL"
-        (path "/2c79a78e-687a-4954-b7b9-175bc3470bd7/cfe63f02-1987-4919-8e32-0515eff710ca"
-          (reference "F1") (unit 1)
-        )
-      )

Commit message: wip kicad
Parts:
- F1: footprint (none) -> Fuse:Fuseholder_Littelfuse_Nano2_154x; Digikey (none) -> F1227CT-ND
Changed lines of the file:
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@@
       (effects (font (size 1.27 1.27)))
     )
-    (property "Footprint" "" (at 101.6 56.388 90)
+    (property "Footprint" "Fuse:Fuseholder_Littelfuse_Nano2_154x" (at 101.6 56.388 90)
       (effects (font (size 1.27 1.27)) hide)
     )
-    (property "Datasheet" "~" (at 101.6 54.61 0)
+    (property "Datasheet" "https://www.littelfuse.com/media?resourcetype=datasheets&itemid=63f61b85-5fc5-4f00-9ca9-8d59a6252d71&filename=littelfuse_fuse_154_154t_154l_154tl_datasheet.pdf" (at 101.6 54.61 0)
       (effects (font (size 1.27 1.27)) hide)
     )
+    (property "Digikey" "F1227CT-ND" (at 101.6 54.61 90)
+      (effects (font (size 1.27 1.27)) hide)
+    )
