File: Kicad/stm32F746 GRBL/stm32F746 GRBL.kicad_sch (KiCad schematic)
At the start: 10 parts, among them CN1 PinHeader_1x08_P2.54mm_Vertic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, CN2 PinHeader_1x06_P2.54mm_Vertic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, CN3 PinHeader_1x10_P2.54mm_Vertic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, CN4 PinHeader_1x08_P2.54mm_Vertic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, J1 Conn_01x03

Commit message: kicad progress
Parts:
- removed J1: Conn_01x03, Connector_PinHeader_2.54mm:PinHeader_1x03_P2.54mm_Vertical, symbol Connector_Generic:Conn_01x03
- added A6: TMC2130_Breakout_TMC2130, stm32F746 GRBL:TMC2130_Breakout-16_15.2x20.3mm, symbol Driver_Motor:Pololu_Breakout_A4988
- added C1, C2, C3: 100nF, symbol Device:C
- added C4, C5, C6, C7, C8, C9: 100uF 50V, Capacitor_SMD:CP_Elec_10x10.5, symbol Device:C_Polarized
- added J1: X-Axis, Connector_JST:JST_XH_B4B-XH-A_1x04_P2.50mm_Vertical, symbol Connector_Generic:Conn_01x04
- added J10, J11, J12, J13, J8, J9: Conn_01x04, Connector_JST:JST_XH_B4B-XH-A_1x04_P2.50mm_Vertical, symbol Connector_Generic:Conn_01x04
- added J2: Y-Axis, Connector_JST:JST_XH_B4B-XH-A_1x04_P2.50mm_Vertical, symbol Connector_Generic:Conn_01x04
- added J3: Z-Axis, Connector_JST:JST_XH_B4B-XH-A_1x04_P2.50mm_Vertical, symbol Connector_Generic:Conn_01x04
- added J4: A-Axis, Connector_JST:JST_XH_B4B-XH-A_1x04_P2.50mm_Vertical, symbol Connector_Generic:Conn_01x04
- added J5: B-Axis, Connector_JST:JST_XH_B4B-XH-A_1x04_P2.50mm_Vertical, symbol Connector_Generic:Conn_01x04
- added J6: C-Axis, Connector_JST:JST_XH_B4B-XH-A_1x04_P2.50mm_Vertical, symbol Connector_Generic:Conn_01x04
- added J7: Screw_Terminal_01x04, Connector_Phoenix_MSTB:PhoenixContact_MSTBA_2,5_4-G-5,08_1x04_P5.08mm_Horizontal, symbol Connector:Screw_Terminal_01x04
- added R1, R10, R11, R12, R13, R14, R15, R16, R17, R18, R19, R2, R20, R21, R22, R3, R4, R5, R6, R7, R8, R9: 100, symbol Device:R
- added U1: 74HCT244, symbol 74xx:74HCT244
- added U2, U4: MCP23008-xSO, Package_SO:SOIC-18W_7.5x11.6mm_P1.27mm, symbol Interface_Expansion:MCP23008-xSO
- added U3: 24LC64, Package_SO:SOIC-8_3.9x4.9mm_P1.27mm, symbol Memory_EEPROM:24LC64
Connections:
- net +3.3V: now also C1.2, C2.1, C3.1, U2.18 (VDD), U3.7 (WP), U3.8 (VCC), U4.18 (VDD), U4.5 (A0)
- net GND: now also A6.1 (GND), A6.7 (GND), C1.1, C2.2, C3.2, C4.2, C5.2, C6.2, C7.2, C8.2, C9.2, J7.4 (Pin_4), U2.3 (A2), U2.4 (A1), U2.5 (A0), U2.9 (VSS), U3.1 (A0), U3.2 (A1), U3.3 (A2), U3.4 (GND), U4.3 (A2), U4.4 (A1), U4.9 (VSS)
- net at CN4.1 (Pin_1): now also R14.1
- net at CN4.2 (Pin_2): now also R13.1
- net at CN4.3 (Pin_3): now also R12.1
- net at CN4.4 (Pin_4): now also R11.1
- net at CN4.5 (Pin_5): now also R10.1
- net at CN4.6 (Pin_6): now also R9.1
- net at CN4.7 (Pin_7): now also R8.1
- net at CN4.8 (Pin_8): now also R7.1
- net at CN2.1 (Pin_1): now also R15.2
- net at CN2.2 (Pin_2): now also R16.1
- net at CN2.3 (Pin_3): now also R17.1
- net at CN2.4 (Pin_4): now also R18.1
- net at CN2.5 (Pin_5): now also R19.1
- net at CN2.6 (Pin_6): now also R20.1
- net RESET: now reaches CN1.3 (Pin_3)
- net RESET: now also U2.6 (~{RESET}), U4.6 (~{RESET})
- net at A1.2 (VDD), A2.2 (VDD), A3.2 (VDD)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: now also A6.2 (VDD)
- net at A2.3 (1B): now also J9.4 (Pin_4)
- net at A2.4 (1A): now also J9.3 (Pin_3)
- net at A2.5 (2A): now also J9.2 (Pin_2)
- net at A2.6 (2B): now also J9.1 (Pin_1)
- net Vdrive: now reaches A2.8 (VMOT)
- net Vdrive: now also A1.8 (VMOT), A3.8 (VMOT), A4.8 (VMOT), A5.8 (VMOT), A6.8 (VMOT), C4.1, C5.1, C6.1, C7.1, C8.1, C9.1, J7.1 (Pin_1)
- net at A5.3 (1B): now also J12.4 (Pin_4)
- net at A5.4 (1A): now also J12.3 (Pin_3)
- net at A5.5 (2A): now also J12.2 (Pin_2)
- net at A5.6 (2B): now also J12.1 (Pin_1)
- net at A4.3 (1B): now also J11.4 (Pin_4)
- net at A4.4 (1A): now also J11.3 (Pin_3)
- net at A4.5 (2A): now also J11.2 (Pin_2)
- net at A4.6 (2B): now also J11.1 (Pin_1)
- net at A3.3 (1B): now also J10.4 (Pin_4)
- net at A3.4 (1A): now also J10.3 (Pin_3)
- net at A3.5 (2A): now also J10.2 (Pin_2)
- net at A3.6 (2B): now also J10.1 (Pin_1)
- net at CN3.1 (Pin_1): now also R6.1
- net at CN3.10 (Pin_10): now also R21.2
- net at CN3.2 (Pin_2): now also R5.1
- net at CN3.3 (Pin_3): now also R4.1
- net at CN3.4 (Pin_4): now also R3.1
- net at CN3.5 (Pin_5): now also R2.1
- net at CN3.6 (Pin_6): now also R1.1
- net at CN3.9 (Pin_9): now also R22.2
- net at A1.3 (1B): now also J8.4 (Pin_4)
- net at A1.4 (1A): now also J8.3 (Pin_3)
- net at A1.5 (2A): now also J8.2 (Pin_2)
- net at A1.6 (2B): now also J8.1 (Pin_1)
- new net: A6.3 (1B), J13.4 (Pin_4)
- new net: A6.4 (1A), J13.3 (Pin_3)
- new net: A6.5 (2A), J13.2 (Pin_2)
- new net: A6.6 (2B), J13.1 (Pin_1)
- new net A-DIR: R16.2
- new net A-STEP: R17.2
- new net AIR: U4.17 (GP7)
- new net COOLANT: U4.10 (GP0)
- new net ENABLE: R15.1
- new net HOLD: U2.10 (GP0)
- new net I2C_SCL: R21.1, U2.1 (SCL), U3.6 (SCL), U4.1 (SCL)
- new net I2C_SDA: R22.1, U2.2 (SDA), U3.5 (SDA), U4.2 (SDA)
- new net INPUT_INT: U2.8 (INT), U4.8 (INT)
- new net PROBE: U2.15 (GP5)
- new net SAFETY_DOOR: U2.17 (GP7)
- new net SLAVE-DIR: R19.2
- new net SLAVE-STEP: R20.2
- new net SPINDLE_DIR: U4.15 (GP5)
Other:
- moved on the sheet: A2, A3, A4, A5, CN1, CN2, CN3, CN4

Commit message: kicad
Parts:
- removed A1, A2, A3, A4, A5, A6: TMC2130_Breakout_TMC2130, stm32F746 GRBL:TMC2130_Breakout-16_15.2x20.3mm, symbol Driver_Motor:Pololu_Breakout_A4988
- removed C1, C2, C3: 100nF, symbol Device:C
- removed C4, C5, C6, C7, C8, C9: 100uF 50V, Capacitor_SMD:CP_Elec_10x10.5, symbol Device:C_Polarized
- removed CN1, CN4: PinHeader_1x08_P2.54mm_Vertical, Connector_PinHeader_2.54mm:PinHeader_1x08_P2.54mm_Vertical, symbol Connector_Generic:Conn_01x08
- removed CN2: PinHeader_1x06_P2.54mm_Vertical, Connector_PinHeader_2.54mm:PinHeader_1x06_P2.54mm_Vertical, symbol Connector_Generic:Conn_01x06
- removed CN3: PinHeader_1x10_P2.54mm_Vertical, Connector_PinHeader_2.54mm:PinHeader_1x10_P2.54mm_Vertical, symbol Connector_Generic:Conn_01x10
- removed J1: X-Axis, Connector_JST:JST_XH_B4B-XH-A_1x04_P2.50mm_Vertical, symbol Connector_Generic:Conn_01x04
- removed J10, J11, J12, J13, J8, J9: Conn_01x04, Connector_JST:JST_XH_B4B-XH-A_1x04_P2.50mm_Vertical, symbol Connector_Generic:Conn_01x04
- removed J2: Y-Axis, Connector_JST:JST_XH_B4B-XH-A_1x04_P2.50mm_Vertical, symbol Connector_Generic:Conn_01x04
- removed J3: Z-Axis, Connector_JST:JST_XH_B4B-XH-A_1x04_P2.50mm_Vertical, symbol Connector_Generic:Conn_01x04
- removed J4: A-Axis, Connector_JST:JST_XH_B4B-XH-A_1x04_P2.50mm_Vertical, symbol Connector_Generic:Conn_01x04
- removed J5: B-Axis, Connector_JST:JST_XH_B4B-XH-A_1x04_P2.50mm_Vertical, symbol Connector_Generic:Conn_01x04
- removed J6: C-Axis, Connector_JST:JST_XH_B4B-XH-A_1x04_P2.50mm_Vertical, symbol Connector_Generic:Conn_01x04
- removed J7: Screw_Terminal_01x04, Connector_Phoenix_MSTB:PhoenixContact_MSTBA_2,5_4-G-5,08_1x04_P5.08mm_Horizontal, symbol Connector:Screw_Terminal_01x04
- removed R1, R10, R11, R12, R13, R14, R15, R16, R17, R18, R19, R2, R20, R21, R22, R3, R4, R5, R6, R7, R8, R9: 100, symbol Device:R
- removed U1: 74HCT244, symbol 74xx:74HCT244
- removed U2, U4: MCP23008-xSO, Package_SO:SOIC-18W_7.5x11.6mm_P1.27mm, symbol Interface_Expansion:MCP23008-xSO
- removed U3: 24LC64, Package_SO:SOIC-8_3.9x4.9mm_P1.27mm, symbol Memory_EEPROM:24LC64
Connections:
- no-connect marks 4 -> 0
Other:
- added sheet Arduino Connector (STM32_Arduino connector.kicad_sch)
- added sheet Driver (Driver.kicad_sch)
- added sheet IO_Expansion (IO_expansion.kicad_sch)
- added sheet Input (Input.kicad_sch)
- added sheet Output (Output.kicad_sch)
- added sheet Power (Power.kicad_sch)

Commit message: wip
Changed lines of the file:
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@@
 (kicad_sch (version 20230121) (generator eeschema)
   (paper "A4")
-  (sheet (at 34.29 25.4) (size 34.29 36.83) (fields_autoplaced)
+  (sheet (at 38.1 25.4) (size 25.4 25.4) (fields_autoplaced)
     (stroke (width 0.1524) (type solid))
     (fill (color 0 0 0 0.0000))
-    (property "Sheetname" "Arduino Connector" (at 34.29 24.6884 0)
+    (property "Sheetname" "Arduino Connector" (at 38.1 24.6884 0)
       (effects (font (size 1.27 1.27)) (justify left bottom))
     )
-    (property "Sheetfile" "STM32_Arduino connector.kicad_sch" (at 34.29 62.8146 0)
+    (property "Sheetfile" "STM32_Arduino connector.kicad_sch" (at 38.1 51.3846 0)
       (effects (font (size 1.27 1.27)) (justify left top))
     )
@@
     )
   )
-  (sheet (at 109.22 74.93) (size 34.29 36.83) (fields_autoplaced)
+  (sheet (at 88.9 63.5) (size 25.4 25.4) (fields_autoplaced)
     (stroke (width 0.1524) (type solid))
     (fill (color 0 0 0 0.0000))
-    (property "Sheetname" "IO_Expansion" (at 109.22 74.2184 0)
+    (property "Sheetname" "IO_Expansion" (at 88.9 62.7884 0)
       (effects (font (size 1.27 1.27)) (justify left bottom))
     )
-    (property "Sheetfile" "IO_expansion.kicad_sch" (at 109.22 112.3446 0)
+    (property "Sheetfile" "IO_expansion.kicad_sch" (at 88.9 89.4846 0)
       (effects (font (size 1.27 1.27)) (justify left top))
     )
@@
     )
   )
-  (sheet (at 34.29 74.93) (size 34.29 36.83) (fields_autoplaced)
+  (sheet (at 38.1 63.5) (size 25.4 25.4) (fields_autoplaced)
     (stroke (width 0.1524) (type solid))
     (fill (color 0 0 0 0.0000))
-    (property "Sheetname" "Driver" (at 34.29 74.2184 0)
+    (property "Sheetname" "Driver" (at 38.1 62.7884 0)
       (effects (font (size 1.27 1.27)) (justify left bottom))
     )
-    (property "Sheetfile" "Driver.kicad_sch" (at 34.29 112.3446 0)
+    (property "Sheetfile" "Driver.kicad_sch" (at 38.1 89.4846 0)
       (effects (font (size 1.27 1.27)) (justify left top))
     )
@@
     )
   )
-  (sheet (at 111.76 138.43) (size 40.64 41.91) (fields_autoplaced)
+  (sheet (at 88.9 101.6) (size 25.4 22.86) (fields_autoplaced)
     (stroke (width 0.1524) (type solid))
     (fill (color 0 0 0 0.0000))
-    (property "Sheetname" "Input" (at 111.76 137.7184 0)
+    (property "Sheetname" "Input" (at 88.9 100.8884 0)
       (effects (font (size 1.27 1.27)) (justify left bottom))
     )
-    (property "Sheetfile" "Input.kicad_sch" (at 111.76 180.9246 0)
+    (property "Sheetfile" "Input.kicad_sch" (at 88.9 125.0446 0)
       (effects (font (size 1.27 1.27)) (justify left top))
     )
@@
     )
   )
-  (sheet (at 111.76 36.83) (size 31.75 31.75) (fields_autoplaced)
+  (sheet (at 88.9 25.4) (size 25.4 25.4) (fields_autoplaced)
     (stroke (width 0.1524) (type solid))
     (fill (color 0 0 0 0.0000))
-    (property "Sheetname" "Power" (at 111.76 36.1184 0)
+    (property "Sheetname" "Power" (at 88.9 24.6884 0)
       (effects (font (size 1.27 1.27)) (justify left bottom))
     )
-    (property "Sheetfile" "Power.kicad_sch" (at 111.76 69.1646 0)
+    (property "Sheetfile" "Power.kicad_sch" (at 88.9 51.3846 0)
       (effects (font (size 1.27 1.27)) (justify left top))
     )
@@
     )
   )
-  (sheet (at 48.26 140.97) (size 34.29 39.37) (fields_autoplaced)
+  (sheet (at 38.1 101.6) (size 25.4 22.86) (fields_autoplaced)
     (stroke (width 0.1524) (type solid))
     (fill (color 0 0 0 0.0000))
-    (property "Sheetname" "Output" (at 48.26 140.2584 0)
+    (property "Sheetname" "Output" (at 38.1 100.8884 0)
       (effects (font (size 1.27 1.27)) (justify left bottom))
     )
-    (property "Sheetfile" "Output.kicad_sch" (at 48.26 180.9246 0)
+    (property "Sheetfile" "Output.kicad_sch" (at 38.1 125.0446 0)
       (effects (font (size 1.27 1.27)) (justify left top))
     )

Commit message: wip Kicad
Other:
- removed sheet IO_Expansion
Changed lines of the file:
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@@
-    )
-  )
-  (sheet (at 88.9 63.5) (size 25.4 25.4) (fields_autoplaced)
-    (stroke (width 0.1524) (type solid))
-    (fill (color 0 0 0 0.0000))
-    (property "Sheetname" "IO_Expansion" (at 88.9 62.7884 0)
-      (effects (font (size 1.27 1.27)) (justify left bottom))
-    )
-    (property "Sheetfile" "IO_expansion.kicad_sch" (at 88.9 89.4846 0)
-      (effects (font (size 1.27 1.27)) (justify left top))
-    )
-    (instances
-      (project "stm32F746 GRBL"
-        (path "/2c79a78e-687a-4954-b7b9-175bc3470bd7" (page "4"))
-      )
     )
   )
