File: Kicad/stm32F746 GRBL/Input.kicad_sch (KiCad schematic)
At the start: 0 parts

Commit message: wip kicad
Parts:
- added J14, J15: Screw_Terminal_01x09, TerminalBlock_TE-Connectivity:TerminalBlock_TE_282834-9_1x09_P2.54mm_Horizontal, symbol Connector:Screw_Terminal_01x09
- added U5, U6: TLP521-4, Package_SO:SOIC-16_4.55x10.3mm_P1.27mm, symbol Isolator:TLP291-4
Connections:
- new net GND: U5.11, U5.13, U5.15, U5.9, U6.11, U6.13, U6.15, U6.9
- new net GNDPWR: U5.2, U5.4, U5.6, U5.8, U6.2, U6.4, U6.6, U6.8
- new net INPUT_1: U5.16
- new net INPUT_2: U5.14
- new net INPUT_3: U5.12
- new net INPUT_4: U5.10
- new net INPUT_5: U6.16
- new net INPUT_6: U6.14
- new net INPUT_7: U6.12
- new net INPUT_8: U6.10

Commit message: wip
Other:
- moved on the sheet: J14, J15
Changed lines of the file:
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@@
     )
   )
-  (symbol (lib_id "Connector:Screw_Terminal_01x09") (at 25.4 132.08 180) (unit 1)
+  (symbol (lib_id "Connector:Screw_Terminal_01x09") (at 113.03 92.71 180) (unit 1)
     (in_bom yes) (on_board yes) (dnp no) (fields_autoplaced)
-    (property "Reference" "J15" (at 25.4 115.57 0)
+    (property "Reference" "J15" (at 113.03 76.2 0)
       (effects (font (size 1.27 1.27)))
     )
-    (property "Value" "Screw_Terminal_01x09" (at 25.4 118.11 0)
+    (property "Value" "Screw_Terminal_01x09" (at 113.03 78.74 0)
       (effects (font (size 1.27 1.27)))
     )
-    (property "Footprint" "TerminalBlock_TE-Connectivity:TerminalBlock_TE_282834-9_1x09_P2.54mm_Horizontal" (at 25.4 132.08 0)
+    (property "Footprint" "TerminalBlock_TE-Connectivity:TerminalBlock_TE_282834-9_1x09_P2.54mm_Horizontal" (at 113.03 92.71 0)
       (effects (font (size 1.27 1.27)) hide)
     )
-    (property "Datasheet" "~" (at 25.4 132.08 0)
+    (property "Datasheet" "~" (at 113.03 92.71 0)
       (effects (font (size 1.27 1.27)) hide)
     )
@@
     )
   )
-  (symbol (lib_id "Connector:Screw_Terminal_01x09") (at 25.4 99.06 180) (unit 1)
+  (symbol (lib_id "Connector:Screw_Terminal_01x09") (at 27.94 93.98 180) (unit 1)
     (in_bom yes) (on_board yes) (dnp no) (fields_autoplaced)
-    (property "Reference" "J14" (at 25.4 82.55 0)
+    (property "Reference" "J14" (at 27.94 77.47 0)
       (effects (font (size 1.27 1.27)))
     )
-    (property "Value" "Screw_Terminal_01x09" (at 25.4 85.09 0)
+    (property "Value" "Screw_Terminal_01x09" (at 27.94 80.01 0)
       (effects (font (size 1.27 1.27)))
     )
-    (property "Footprint" "TerminalBlock_TE-Connectivity:TerminalBlock_TE_282834-9_1x09_P2.54mm_Horizontal" (at 25.4 99.06 0)
+    (property "Footprint" "TerminalBlock_TE-Connectivity:TerminalBlock_TE_282834-9_1x09_P2.54mm_Horizontal" (at 27.94 93.98 0)
       (effects (font (size 1.27 1.27)) hide)
     )
-    (property "Datasheet" "~" (at 25.4 99.06 0)
+    (property "Datasheet" "~" (at 27.94 93.98 0)
       (effects (font (size 1.27 1.27)) hide)
     )

Commit message: wip Kicad
Parts:
- added C1, C2: 100nF, Capacitor_SMD:C_0805_2012Metric, symbol Device:C
- added RN1, RN2: 4K7, Resistor_THT:R_Array_SIP9, symbol Device:R_Network08_Split
- added U1, U2: MCP23008-xSO, Package_SO:SOIC-18W_7.5x11.6mm_P1.27mm, symbol Interface_Expansion:MCP23008-xSO
- added U7, U8: TLP521-4, Package_SO:SOIC-16_4.55x10.3mm_P1.27mm, symbol Isolator:TLP291-4
- J14: value Screw_Terminal_01x09 -> Input 1-8
- J15: value Screw_Terminal_01x09 -> Input 9-16
Connections:
- net GND: now also J14.1 (Pin_1), J15.1 (Pin_1), C1.2, C2.2, U1.3 (A2), U1.4 (A1), U1.5 (A0), U1.9 (VSS), U2.3 (A2), U2.4 (A1), U2.9 (VSS), U7.11, U7.13, U7.15, U7.9, U8.11, U8.13, U8.15, U8.9
- net INPUT_1: now also RN1.2 (R1.2), U1.10 (GP0)
- net INPUT_2: now also RN1.3 (R2.2), U1.11 (GP1)
- net INPUT_3: now also RN1.4 (R3.2), U1.12 (GP2)
- net INPUT_4: now also RN1.5 (R4.2), U1.13 (GP3)
- net INPUT_5: now also RN1.6 (R5.2), U1.14 (GP4)
- net INPUT_6: now also RN1.7 (R6.2), U1.15 (GP5)
- net INPUT_7: now also RN1.8 (R7.2), U1.16 (GP6)
- net INPUT_8: now also RN1.9 (R8.2), U1.17 (GP7)
- removed net GNDPWR: U5.2, U5.4, U5.6, U5.8, U6.2, U6.4, U6.6, U6.8
- new net +3.3VP: C1.1, C2.1, RN1.1 (R1), RN1.1 (R1), RN1.1 (R1), RN1.1 (R1), RN1.1 (R1), RN1.1 (R1), RN1.1 (R1), RN1.1 (R1), RN2.1 (R1), RN2.1 (R1), RN2.1 (R1), RN2.1 (R1), RN2.1 (R1), RN2.1 (R1), RN2.1 (R1), RN2.1 (R1), U1.18 (VDD), U2.18 (VDD), U2.5 (A0)
- new net I2C_SCL: U1.1 (SCL), U2.1 (SCL)
- new net I2C_SDA: U1.2 (SDA), U2.2 (SDA)
- new net INPUT_10: RN2.3 (R2.2), U2.11 (GP1), U7.14
- new net INPUT_11: RN2.4 (R3.2), U2.12 (GP2), U7.12
- new net INPUT_12: RN2.5 (R4.2), U2.13 (GP3), U7.10
- new net INPUT_13: RN2.6 (R5.2), U2.14 (GP4), U8.16
- new net INPUT_14: RN2.7 (R6.2), U2.15 (GP5), U8.14
- new net INPUT_15: RN2.8 (R7.2), U2.16 (GP6), U8.12
- new net INPUT_16: RN2.9 (R8.2), U2.17 (GP7), U8.10
- new net INPUT_9: RN2.2 (R1.2), U2.10 (GP0), U7.16
- new net INPUT_INT_1: U1.8 (INT)
- new net INPUT_INT_2: U2.8 (INT)
- new net RESET: U1.6 (~{RESET}), U2.6 (~{RESET})
Other:
- note added: "0x20 - 0100(000)x"
- note added: "0x21 - 0100(001)x"
- moved on the sheet: J14, J15, U5A, U5B, U5C, U5D, U6A, U6B, U6C, U6D

Commit message: kicad wip
Parts:
- removed U1, U2: MCP23008-xSO, Package_SO:SOIC-18W_7.5x11.6mm_P1.27mm, symbol Interface_Expansion:MCP23008-xSO
- added RN3, RN4: 390, Package_SO:SOIC-16_4.55x10.3mm_P1.27mm, symbol Device:R_Pack08_Split
- added RN5, RN6: 4K7, Resistor_THT:R_Array_SIP9, symbol Device:R_Network08_Split
- added U1, U2: MCP23008-xSS, Package_SO:SSOP-20_5.3x7.2mm_P0.65mm, symbol Interface_Expansion:MCP23008-xSS
Connections:
- net +3.3VP: now also U1.20 (VDD), U2.20 (VDD), U2.5 (A0)
- net GND: now also J14.9 (Pin_9), J15.9 (Pin_9), U5.2, U5.4, U5.6, U5.8, U6.2, U6.4, U6.6, U6.8, U7.2, U7.4, U7.6, U7.8, U8.2, U8.4, U8.6, U8.8, RN5.1 (R1), RN5.1 (R1), RN5.1 (R1), RN5.1 (R1), RN5.1 (R1), RN5.1 (R1), RN5.1 (R1), RN5.1 (R1), RN6.1 (R1), RN6.1 (R1), RN6.1 (R1), RN6.1 (R1), RN6.1 (R1), RN6.1 (R1), RN6.1 (R1), RN6.1 (R1), U1.3 (A2), U1.4 (A1), U1.5 (A0), U1.9 (VSS), U2.3 (A2), U2.4 (A1), U2.9 (VSS); no longer J14.1 (Pin_1), J15.1 (Pin_1)
- net I2C_SCL: now also U1.1 (SCL), U2.1 (SCL)
- net I2C_SDA: now also U1.2 (SDA), U2.2 (SDA)
- net INPUT_1: now also U1.12 (GP0)
- net INPUT_10: now also U2.13 (GP1)
- net INPUT_11: now also U2.14 (GP2)
- net INPUT_12: now also U2.15 (GP3)
- net INPUT_13: now also U2.16 (GP4)
- net INPUT_14: now also U2.17 (GP5)
- net INPUT_15: now also U2.18 (GP6)
- net INPUT_16: now also U2.19 (GP7)
- net INPUT_2: now also U1.13 (GP1)
- net INPUT_3: now also U1.14 (GP2)
- net INPUT_4: now also U1.15 (GP3)
- net INPUT_5: now also U1.16 (GP4)
- net INPUT_6: now also U1.17 (GP5)
- net INPUT_7: now also U1.18 (GP6)
- net INPUT_8: now also U1.19 (GP7)
- net INPUT_9: now also U2.12 (GP0)
- net INPUT_INT_1: now also U1.8 (INT)
- net INPUT_INT_2: now also U2.8 (INT)
- net RESET: now also U1.6 (~{RESET}), U2.6 (~{RESET})
- net at U8.1: now also RN4.5 (R5.1), RN6.6 (R5.2)
- net at U5.1: now also RN3.1 (R1.1), RN5.2 (R1.2)
- net at U8.5: now also RN4.7 (R7.1), RN6.8 (R7.2)
- net at U7.3: now also RN4.2 (R2.1), RN6.3 (R2.2)
- net at U7.5: now also RN4.3 (R3.1), RN6.4 (R3.2)
- net at U8.3: now also RN4.6 (R6.1), RN6.7 (R6.2)
- net at U6.5: now also RN3.7 (R7.1), RN5.8 (R7.2)
- net at U7.7: now also RN4.4 (R4.1), RN6.5 (R4.2)
- net IN10: now reaches J15.2 (Pin_2)
- net IN10: now also RN4.15 (R2.2)
- net IN11: now reaches J15.3 (Pin_3)
- net IN11: now also RN4.14 (R3.2)
- net IN12: now reaches J15.4 (Pin_4)
- net IN12: now also RN4.13 (R4.2)
- net IN13: now reaches J15.5 (Pin_5)
- net IN13: now also RN4.12 (R5.2)
- net IN14: now reaches J15.6 (Pin_6)
- net IN14: now also RN4.11 (R6.2)
- net IN15: now reaches J15.7 (Pin_7)
- net IN15: now also RN4.10 (R7.2)
- net IN16: now reaches J15.8 (Pin_8)
- net IN16: now also RN4.9 (R8.2)
- net at U5.7: now also RN3.4 (R4.1), RN5.5 (R4.2)
- net at U6.1: now also RN3.5 (R5.1), RN5.6 (R5.2)
- net at U8.7: now also RN4.8 (R8.1), RN6.9 (R8.2)
- net IN2: now reaches J14.2 (Pin_2)
- net IN2: now also RN3.15 (R2.2)
- net IN3: now reaches J14.3 (Pin_3)
- net IN3: now also RN3.14 (R3.2)
- net IN4: now reaches J14.4 (Pin_4)
- net IN4: now also RN3.13 (R4.2)
- net IN5: now reaches J14.5 (Pin_5)
- net IN5: now also RN3.12 (R5.2)
- net IN6: now reaches J14.6 (Pin_6)
- net IN6: now also RN3.11 (R6.2)
- net IN7: now reaches J14.7 (Pin_7)
- net IN7: now also RN3.10 (R7.2)
- net IN8: now reaches J14.8 (Pin_8)
- net IN8: now also RN3.9 (R8.2)
- net at U5.3: now also RN3.2 (R2.1), RN5.3 (R2.2)
- net at U6.7: now also RN3.8 (R8.1), RN5.9 (R8.2)
- net at U7.1: now also RN4.1 (R1.1), RN6.2 (R1.2)
- net at U5.5: now also RN3.3 (R3.1), RN5.4 (R3.2)
- net at U6.3: now also RN3.6 (R6.1), RN5.7 (R6.2)
- new net IN1: J14.1 (Pin_1), RN3.16 (R1.2)
- new net IN9: J15.1 (Pin_1), RN4.16 (R1.2)
Other:
- moved on the sheet: J14, J15
