File: Kicad/stm32F746 GRBL/stm32F746 GRBL.kicad_pcb (KiCad board)
At the start: 2 copper layers, 130 x 80 mm, 14 parts, among them CN1 PinHeader_1x08_P2.54mm_Vertic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, CN2 PinHeader_1x06_P2.54mm_Vertic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, CN3 PinHeader_1x10_P2.54mm_Vertic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, CN4 PinHeader_1x08_P2.54mm_Vertic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, J1 Conn_01x03

Commit message: kicad progress
Parts:
- added A6: TMC2130_Breakout_TMC2130, stm32F746 GRBL:TMC2130_Breakout-16_15.2x20.3mm, F.Cu at (183.2, 94.0)
- added C1: 100nF, Capacitor_SMD:C_0805_2012Metric, F.Cu at (117.5, 110.0)
- added C2: 100nF, Capacitor_SMD:C_0805_2012Metric, F.Cu at (107.7, 80.5)
- added C3: 100nF, Capacitor_SMD:C_0805_2012Metric, F.Cu at (108.0, 98.0)
- added J10: B-Axis, Connector_JST:JST_XH_B4B-XH-A_1x04_P2.50mm_Vertical, F.Cu at (174.8, 63.0)
- added J11: Conn_01x04, Connector_JST:JST_XH_B4B-XH-A_1x04_P2.50mm_Vertical, F.Cu at (127.0, 88.0)
- added J12: C-Axis, Connector_JST:JST_XH_B4B-XH-A_1x04_P2.50mm_Vertical, F.Cu at (152.8, 88.0)
- added J13: Conn_01x04, Connector_JST:JST_XH_B4B-XH-A_1x04_P2.50mm_Vertical, F.Cu at (174.8, 88.0)
- added J2: Conn_01x04, Connector_JST:JST_XH_B4B-XH-A_1x04_P2.50mm_Vertical, F.Cu at (154.5, 126.2)
- added J3: Y-Axis, Connector_JST:JST_XH_B4B-XH-A_1x04_P2.50mm_Vertical, F.Cu at (162.5, 126.2)
- added J4: Conn_01x04, Connector_JST:JST_XH_B4B-XH-A_1x04_P2.50mm_Vertical, F.Cu at (170.5, 126.2)
- added J5: Z-Axis, Connector_JST:JST_XH_B4B-XH-A_1x04_P2.50mm_Vertical, F.Cu at (178.5, 126.2)
- added J6: Conn_01x04, Connector_JST:JST_XH_B4B-XH-A_1x04_P2.50mm_Vertical, F.Cu at (186.5, 126.2)
- added J7: Screw_Terminal_01x04, Connector_Phoenix_MSTB:PhoenixContact_MSTBA_2,5_4-G-5,08_1x04_P5.08mm_Horizontal, F.Cu at (91.4, 122.0)
- added J8: A-Axis, Connector_JST:JST_XH_B4B-XH-A_1x04_P2.50mm_Vertical, F.Cu at (127.0, 63.0)
- added J9: Conn_01x04, Connector_JST:JST_XH_B4B-XH-A_1x04_P2.50mm_Vertical, F.Cu at (152.8, 63.0)
- added U2: MCP23008-xSO, Package_SO:SOIC-18W_7.5x11.6mm_P1.27mm, F.Cu at (106.0, 88.0)
- added U3: 24LC64, Package_SO:SOIC-8_3.9x4.9mm_P1.27mm, F.Cu at (119.5, 114.1)
- added U4: MCP23008-xSO, Package_SO:SOIC-18W_7.5x11.6mm_P1.27mm, F.Cu at (106.0, 107.0)
- J1: value Conn_01x03 -> X-Axis; footprint Connector_PinHeader_2.54mm:PinHeader_1x03_P2.54mm_Vertical -> Connector_JST:JST_XH_B4B-XH-A_1x04_P2.50mm_Vertical
- moved A3 86.5 mm to (183.4, 69.0)
- moved J1 45.9 mm to (146.5, 126.2), turned to 90 degrees
- moved A5 38.9 mm to (161.4, 94.0)
- moved A1 35.6 mm to (135.6, 69.0)
- moved A2 31.5 mm to (161.4, 69.0)
- moved A4 5.75 mm to (135.4, 94.0)
Connections:
- A1 pad 15: unconnected-(A1-STEP-Pad15) -> /X-STEP
- A1 pad 16: unconnected-(A1-DIR-Pad16) -> /X-DIR
- A1 pad 3: unconnected-(A1-1B-Pad3) -> Net-(A1-1B)
- A1 pad 4: unconnected-(A1-1A-Pad4) -> Net-(A1-1A)
- A1 pad 5: unconnected-(A1-2A-Pad5) -> Net-(A1-2A)
- A1 pad 6: unconnected-(A1-2B-Pad6) -> Net-(A1-2B)
- A1 pad 8: unconnected-(A1-VMOT-Pad8) -> Vdrive
- A1 pad 9: unconnected-(A1-~{ENABLE}-Pad9) -> /ENABLE
- A2 pad 15: unconnected-(A2-STEP-Pad15) -> /Y-STEP
- A2 pad 16: unconnected-(A2-DIR-Pad16) -> /Y-DIR
- A2 pad 3: unconnected-(A2-1B-Pad3) -> Net-(A2-1B)
- A2 pad 4: unconnected-(A2-1A-Pad4) -> Net-(A2-1A)
- A2 pad 5: unconnected-(A2-2A-Pad5) -> Net-(A2-2A)
- A2 pad 6: unconnected-(A2-2B-Pad6) -> Net-(A2-2B)
- A2 pad 8: unconnected-(A2-VMOT-Pad8) -> Vdrive
- A2 pad 9: unconnected-(A2-~{ENABLE}-Pad9) -> /ENABLE
- A3 pad 15: unconnected-(A3-STEP-Pad15) -> /Z-STEP
- A3 pad 16: unconnected-(A3-DIR-Pad16) -> /Z-DIR
- A3 pad 3: unconnected-(A3-1B-Pad3) -> Net-(A3-1B)
- A3 pad 4: unconnected-(A3-1A-Pad4) -> Net-(A3-1A)
- A3 pad 5: unconnected-(A3-2A-Pad5) -> Net-(A3-2A)
- A3 pad 6: unconnected-(A3-2B-Pad6) -> Net-(A3-2B)
- A3 pad 8: unconnected-(A3-VMOT-Pad8) -> Vdrive
- A3 pad 9: unconnected-(A3-~{ENABLE}-Pad9) -> /ENABLE
- A4 pad 15: unconnected-(A4-STEP-Pad15) -> /A-STEP
- A4 pad 16: unconnected-(A4-DIR-Pad16) -> /A-DIR
- A4 pad 3: unconnected-(A4-1B-Pad3) -> Net-(A4-1B)
- A4 pad 4: unconnected-(A4-1A-Pad4) -> Net-(A4-1A)
- A4 pad 5: unconnected-(A4-2A-Pad5) -> Net-(A4-2A)
- A4 pad 6: unconnected-(A4-2B-Pad6) -> Net-(A4-2B)
- A4 pad 8: unconnected-(A4-VMOT-Pad8) -> Vdrive
- A4 pad 9: unconnected-(A4-~{ENABLE}-Pad9) -> /ENABLE
- A5 pad 15: unconnected-(A5-STEP-Pad15) -> /B-STEP
- A5 pad 16: unconnected-(A5-DIR-Pad16) -> /B-DIR
- A5 pad 3: unconnected-(A5-1B-Pad3) -> Net-(A5-1B)
- A5 pad 4: unconnected-(A5-1A-Pad4) -> Net-(A5-1A)
- A5 pad 5: unconnected-(A5-2A-Pad5) -> Net-(A5-2A)
- A5 pad 6: unconnected-(A5-2B-Pad6) -> Net-(A5-2B)
- A5 pad 8: unconnected-(A5-VMOT-Pad8) -> Vdrive
- A5 pad 9: unconnected-(A5-~{ENABLE}-Pad9) -> /ENABLE
- CN1 pad 3: unconnected-(CN1-Pin_3-Pad3) -> /RESET
- CN2 pad 1: unconnected-(CN2-Pin_1-Pad1) -> Net-(CN2-Pin_1)
- CN2 pad 2: unconnected-(CN2-Pin_2-Pad2) -> Net-(CN2-Pin_2)
- CN2 pad 3: unconnected-(CN2-Pin_3-Pad3) -> Net-(CN2-Pin_3)
- CN2 pad 4: unconnected-(CN2-Pin_4-Pad4) -> Net-(CN2-Pin_4)
- CN2 pad 5: unconnected-(CN2-Pin_5-Pad5) -> Net-(CN2-Pin_5)
- CN2 pad 6: unconnected-(CN2-Pin_6-Pad6) -> Net-(CN2-Pin_6)
- CN3 pad 1: unconnected-(CN3-Pin_1-Pad1) -> Net-(CN3-Pin_1)
- CN3 pad 10: unconnected-(CN3-Pin_10-Pad10) -> Net-(CN3-Pin_10)
- CN3 pad 2: unconnected-(CN3-Pin_2-Pad2) -> Net-(CN3-Pin_2)
- CN3 pad 3: unconnected-(CN3-Pin_3-Pad3) -> Net-(CN3-Pin_3)
- CN3 pad 4: unconnected-(CN3-Pin_4-Pad4) -> Net-(CN3-Pin_4)
- CN3 pad 5: unconnected-(CN3-Pin_5-Pad5) -> Net-(CN3-Pin_5)
- CN3 pad 6: unconnected-(CN3-Pin_6-Pad6) -> Net-(CN3-Pin_6)
- CN3 pad 9: unconnected-(CN3-Pin_9-Pad9) -> Net-(CN3-Pin_9)
- CN4 pad 1: unconnected-(CN4-Pin_1-Pad1) -> Net-(CN4-Pin_1)
- CN4 pad 2: unconnected-(CN4-Pin_2-Pad2) -> Net-(CN4-Pin_2)
- CN4 pad 3: unconnected-(CN4-Pin_3-Pad3) -> Net-(CN4-Pin_3)
- CN4 pad 4: unconnected-(CN4-Pin_4-Pad4) -> Net-(CN4-Pin_4)
- CN4 pad 5: unconnected-(CN4-Pin_5-Pad5) -> Net-(CN4-Pin_5)
- CN4 pad 6: unconnected-(CN4-Pin_6-Pad6) -> Net-(CN4-Pin_6)
- CN4 pad 7: unconnected-(CN4-Pin_7-Pad7) -> Net-(CN4-Pin_7)
- CN4 pad 8: unconnected-(CN4-Pin_8-Pad8) -> Net-(CN4-Pin_8)
- J1 pad 1: +3.3V -> /ENABLE
- J1 pad 2: Net-(A1-VDD) -> /X-STEP
- J1 pad 3: +5V -> /X-DIR
Other:
- outline, holes or cut-outs redrawn

Commit message: kicad
Parts:
- added Q1: STD30NF06, Package_TO_SOT_SMD:TO-252-2, F.Cu at (-55.9, 16.1)
- added Q2: STD30NF06, Package_TO_SOT_SMD:TO-252-2, F.Cu at (-55.9, 24.2)
- added Q3: STD30NF06, Package_TO_SOT_SMD:TO-252-2, F.Cu at (-55.9, 32.2)
- added RN1: 100, Package_SO:SOIC-16W-12_7.5x10.3mm_P1.27mm, F.Cu at (-71.6, 33.2)
- added U1: MCP23008-xSO, Package_SO:SOIC-18W_7.5x11.6mm_P1.27mm, F.Cu at (-71.3, 18.6)
- J11: renamed from J12; value C-Axis -> Conn_01x04
- J2: value Conn_01x04 -> Y-Axis
- J3: value Y-Axis -> Z-Axis
- J4: value Conn_01x04 -> A-Axis
- J5: value Z-Axis -> B-Axis
- J6: value Conn_01x04 -> C-Axis
- J7: renamed from J8; value A-Axis -> Conn_01x04
- J9: renamed from J10; value B-Axis -> Conn_01x04
- renumbered J11 to J10, J13 to J12, J7 to J13, J9 to J8
Connections:
- net /HOLD renamed /IO_Expansion/ENABLE
- net /SAFETY_DOOR renamed /IO_Expansion/AIR
- net /X-DIR renamed /Driver/X-DIR
- net /X-STEP renamed /Driver/X-STEP
- net /Y-DIR renamed /Driver/Z-DIR
- net /Y-STEP renamed /Driver/Z-STEP
- A1 pad 2: Net-(A1-VDD) -> unconnected-(A1-VDD-Pad2)
- A1 pad 9: /ENABLE -> /Driver/ENABLE
- A2 pad 2: Net-(A1-VDD) -> unconnected-(A2-VDD-Pad2)
- A2 pad 9: /ENABLE -> /Driver/ENABLE
- A3 pad 15: /Z-STEP -> /Driver/Y-STEP
- A3 pad 16: /Z-DIR -> /Driver/Y-DIR
- A3 pad 2: Net-(A1-VDD) -> unconnected-(A3-VDD-Pad2)
- A3 pad 9: /ENABLE -> /Driver/ENABLE
- A4 pad 15: /A-STEP -> /Driver/A-STEP
- A4 pad 16: /A-DIR -> /Driver/A-DIR
- A4 pad 2: Net-(A1-VDD) -> unconnected-(A4-VDD-Pad2)
- A4 pad 9: /ENABLE -> /Driver/ENABLE
- A5 pad 15: /B-STEP -> /Driver/B-STEP
- A5 pad 16: /B-DIR -> /Driver/B-DIR
- A5 pad 2: Net-(A1-VDD) -> unconnected-(A5-VDD-Pad2)
- A5 pad 9: /ENABLE -> /Driver/ENABLE
- A6 pad 15: /C-STEP -> /Driver/C-STEP
- A6 pad 16: /C-DIR -> /Driver/C-DIR
- A6 pad 2: Net-(A1-VDD) -> unconnected-(A6-VDD-Pad2)
- A6 pad 9: /ENABLE -> /Driver/ENABLE
- C1 pad 1: GND -> +3.3V
- C1 pad 2: +3.3V -> GND
- C3 pad 1: +3.3V -> GND
- C3 pad 2: GND -> +3.3V
- CN1 pad 3: /RESET -> /Arduino Connector/RESET
- CN3 pad 1: Net-(CN3-Pin_1) -> unconnected-(CN3-Pin_1-Pad1)
- CN3 pad 3: Net-(CN3-Pin_3) -> unconnected-(CN3-Pin_3-Pad3)
- CN3 pad 5: Net-(CN3-Pin_5) -> unconnected-(CN3-Pin_5-Pad5)
- J1 pad 1: /ENABLE -> /Driver/ENABLE
- J10 pad 1: Net-(A5-2B) -> Net-(A4-2B)
- J10 pad 2: Net-(A5-2A) -> Net-(A4-2A)
- J10 pad 3: Net-(A5-1A) -> Net-(A4-1A)
- J10 pad 4: Net-(A5-1B) -> Net-(A4-1B)
- J11 pad 1: /ENABLE -> Net-(A5-2B)
- J11 pad 2: /C-STEP -> Net-(A5-2A)
- J11 pad 3: /C-DIR -> Net-(A5-1A)
- J11 pad 4: GND -> Net-(A5-1B)
- J13 pad 1: unconnected-(J7-Pin_1-Pad1) -> Vdrive
- J2 pad 1: Net-(A1-2B) -> /Driver/ENABLE
- J2 pad 2: Net-(A1-2A) -> /Driver/Y-STEP
- J2 pad 3: Net-(A1-1A) -> /Driver/Y-DIR
- J2 pad 4: Net-(A1-1B) -> GND
- J3 pad 1: /ENABLE -> /Driver/ENABLE
- J4 pad 1: Net-(A2-2B) -> /Driver/ENABLE
- J4 pad 2: Net-(A2-2A) -> /Driver/A-STEP
- J4 pad 3: Net-(A2-1A) -> /Driver/A-DIR
- J4 pad 4: Net-(A2-1B) -> GND
- J5 pad 1: /ENABLE -> /Driver/ENABLE
- J5 pad 2: /Z-STEP -> /Driver/B-STEP
- J5 pad 3: /Z-DIR -> /Driver/B-DIR
- J6 pad 1: Net-(A3-2B) -> /Driver/ENABLE
- J6 pad 2: Net-(A3-2A) -> /Driver/C-STEP
- J6 pad 3: Net-(A3-1A) -> /Driver/C-DIR
- J6 pad 4: Net-(A3-1B) -> GND
- J7 pad 1: /ENABLE -> Net-(A1-2B)
- J7 pad 2: /A-STEP -> Net-(A1-2A)
- J7 pad 3: /A-DIR -> Net-(A1-1A)
- J7 pad 4: GND -> Net-(A1-1B)
- J8 pad 1: Net-(A4-2B) -> Net-(A2-2B)
- J8 pad 2: Net-(A4-2A) -> Net-(A2-2A)
- J8 pad 3: Net-(A4-1A) -> Net-(A2-1A)
- J8 pad 4: Net-(A4-1B) -> Net-(A2-1B)
- J9 pad 1: /ENABLE -> Net-(A3-2B)
- J9 pad 2: /B-STEP -> Net-(A3-2A)
- J9 pad 3: /B-DIR -> Net-(A3-1A)
- J9 pad 4: GND -> Net-(A3-1B)
- U2 pad 1: /I2C_SCL -> /IO_Expansion/I2C_SCL
- U2 pad 11: unconnected-(U2-GP1-Pad11) -> /IO_Expansion/SPINDLE_DIR
- U2 pad 12: unconnected-(U2-GP2-Pad12) -> /IO_Expansion/SPINDLE_EN
- U2 pad 13: unconnected-(U2-GP3-Pad13) -> /IO_Expansion/COOLANT
- U2 pad 15: /PROBE -> unconnected-(U2-GP5-Pad15)
- U2 pad 2: /I2C_SDA -> /IO_Expansion/I2C_SDA
- U2 pad 5: GND -> +3.3V
- U2 pad 6: /RESET -> /IO_Expansion/RESET
- U2 pad 8: /INPUT_INT -> unconnected-(U2-INT-Pad8)
- U3 pad 5: /I2C_SDA -> /Arduino Connector/I2C_SDA
- U3 pad 6: /I2C_SCL -> /Arduino Connector/I2C_SCL

Commit message: wip kicad
Parts:
- added J14: Screw_Terminal_01x09, TerminalBlock_TE-Connectivity:TerminalBlock_TE_282834-9_1x09_P2.54mm_Horizontal, F.Cu at (81.8, 95.0)
- added J15: Screw_Terminal_01x09, TerminalBlock_TE-Connectivity:TerminalBlock_TE_282834-9_1x09_P2.54mm_Horizontal, F.Cu at (81.8, 70.5)
- added J16: Screw_Terminal_01x09, TerminalBlock_TE-Connectivity:TerminalBlock_TE_282834-9_1x09_P2.54mm_Horizontal, F.Cu at (109.3, 63.0)
- added RN2: 100, Package_SO:SOIC-16W_5.3x10.2mm_P1.27mm, B.Cu at (149.8, 100.3)
- added RN3: 100, Package_SO:SOIC-16W_5.3x10.2mm_P1.27mm, B.Cu at (149.8, 75.2)
- added U5: TLP521-4, Package_SO:SOIC-16_4.55x10.3mm_P1.27mm, F.Cu at (92.6, 73.0)
- added U6: TLP521-4, Package_SO:SOIC-16_4.55x10.3mm_P1.27mm, F.Cu at (92.5, 86.8)
- RN1: footprint Package_SO:SOIC-16W-12_7.5x10.3mm_P1.27mm -> Package_SO:SOIC-16W_5.3x10.2mm_P1.27mm; moved to B.Cu
- U4: value MCP23008-xSO -> XTR115U; footprint Package_SO:SOIC-18W_7.5x11.6mm_P1.27mm -> Package_SO:SOIC-8_3.9x4.9mm_P1.27mm
- moved RN1 247.0 mm to (171.8, 75.3), turned to -90 degrees
- moved U1 188.2 mm to (107.8, 76.3), turned to 180 degrees
- moved Q1 171.6 mm to (49.0, 151.9)
- moved Q2 171.6 mm to (49.0, 159.9)
- moved Q3 171.6 mm to (49.0, 168.0)
- moved C2 36.0 mm to (120.3, 114.2)
- moved C3 34.3 mm to (134.3, 120.0)
- moved U4 34.2 mm to (132.2, 129.0)
- moved U2 12.7 mm to (108.0, 100.5)
- moved C1 10.9 mm to (120.0, 120.7)
- moved U3 10.9 mm to (122.0, 124.8)
Connections:
- net /IO_Expansion/AIR renamed INPUT_16
- net /IO_Expansion/COOLANT renamed INPUT_12
- net /IO_Expansion/ENABLE renamed INPUT_9
- net /IO_Expansion/SPINDLE_DIR renamed INPUT_10
- net /IO_Expansion/SPINDLE_EN renamed INPUT_11
- U1 pad 10: /IO_Expansion/HOLD -> INPUT_1
- U1 pad 11: unconnected-(U1-GP1-Pad11) -> INPUT_2
- U1 pad 12: unconnected-(U1-GP2-Pad12) -> INPUT_3
- U1 pad 13: unconnected-(U1-GP3-Pad13) -> INPUT_4
- U1 pad 14: unconnected-(U1-GP4-Pad14) -> INPUT_5
- U1 pad 15: /IO_Expansion/PROBE -> INPUT_6
- U1 pad 16: unconnected-(U1-GP6-Pad16) -> INPUT_7
- U1 pad 17: /IO_Expansion/SAFETY_DOOR -> INPUT_8
- U2 pad 14: unconnected-(U2-GP4-Pad14) -> INPUT_13
- U2 pad 15: unconnected-(U2-GP5-Pad15) -> INPUT_14
- U2 pad 16: unconnected-(U2-GP6-Pad16) -> INPUT_15
- U2 pad 8: unconnected-(U2-INT-Pad8) -> /IO_Expansion/INPUT_INT
- U4 pad 1: /I2C_SCL -> unconnected-(U4-VREF-Pad1)
- U4 pad 2: /I2C_SDA -> unconnected-(U4-IIN-Pad2)
- U4 pad 3: GND -> unconnected-(U4-IRET-Pad3)
- U4 pad 4: GND -> unconnected-(U4-IO-Pad4)
- U4 pad 5: +3.3V -> unconnected-(U4-E-Pad5)
- U4 pad 6: /RESET -> unconnected-(U4-B-Pad6)

Commit message: wip
Parts:
- removed RN1, RN2, RN3: 100, Package_SO:SOIC-16W_5.3x10.2mm_P1.27mm
- added D1: 2BZX84C3V9, Package_TO_SOT_SMD:SOT-23, B.Cu at (129.2, 74.0)
- added D2: 2BZX84C3V9, Package_TO_SOT_SMD:SOT-23, B.Cu at (155.1, 73.1)
- added D3: 2BZX84C3V9, Package_TO_SOT_SMD:SOT-23, B.Cu at (176.6, 73.3)
- added D4: 2BZX84C3V9, Package_TO_SOT_SMD:SOT-23, B.Cu at (129.2, 97.9)
- added D5: 2BZX84C3V9, Package_TO_SOT_SMD:SOT-23, B.Cu at (154.8, 98.2)
- added D6: 2BZX84C3V9, Package_TO_SOT_SMD:SOT-23, B.Cu at (177.0, 98.4)
- added D7: BZX84Cxx, Package_TO_SOT_SMD:SOT-23, B.Cu at (194.7, 94.2)
- added PS1: B0503LS-1WR3, stm32F746 GRBL:CONV_B0503LS-1WR3, F.Cu at (126.2, 129.0)
- added R1: 270, Resistor_SMD:R_0805_2012Metric, B.Cu at (128.2, 77.8)
- added R10: 270, Resistor_SMD:R_0805_2012Metric, B.Cu at (156.0, 102.2)
- added R11: 270, Resistor_SMD:R_0805_2012Metric, B.Cu at (175.5, 102.4)
- added R12: 270, Resistor_SMD:R_0805_2012Metric, B.Cu at (177.8, 102.4)
- added R13: 270, Resistor_SMD:R_0805_2012Metric, B.Cu at (194.0, 99.8)
- added R2: 270, Resistor_SMD:R_0805_2012Metric, B.Cu at (130.2, 77.8)
- added R3: 270, Resistor_SMD:R_0805_2012Metric, B.Cu at (153.2, 77.2)
- added R4: 270, Resistor_SMD:R_0805_2012Metric, B.Cu at (156.0, 77.2)
- added R5: 270, Resistor_SMD:R_0805_2012Metric, B.Cu at (175.5, 77.1)
- added R6: 270, Resistor_SMD:R_0805_2012Metric, B.Cu at (177.5, 77.1)
- added R7: 270, Resistor_SMD:R_0805_2012Metric, B.Cu at (128.2, 101.7)
- added R8: 270, Resistor_SMD:R_0805_2012Metric, B.Cu at (130.2, 101.9)
- added R9: 270, Resistor_SMD:R_0805_2012Metric, B.Cu at (153.8, 102.4)
- added U7: 74AHCT1G125, Package_TO_SOT_SMD:SOT-353_SC-70-5, B.Cu at (195.4, 106.7)
- moved U4 50.4 mm to (90.5, 100.8)
- moved C3 38.0 mm to (97.2, 111.8)
- moved U3 34.4 mm to (91.0, 109.9)
- moved C2 27.3 mm to (97.5, 99.2)
- moved C1 27.3 mm to (97.5, 105.2)
- moved U2 4.03 mm to (107.5, 104.5)
- moved U1 3.35 mm to (104.8, 75.0)
- moved U5 2.07 mm to (91.2, 74.6), turned to 0 degrees
- moved U6 1.46 mm to (91.2, 87.5), turned to 0 degrees
Connections:
- CN2 pad 1: Net-(CN2-Pin_1) -> CPU_A-DIR
- CN2 pad 2: Net-(CN2-Pin_2) -> CPU_B-DIR
- CN2 pad 3: Net-(CN2-Pin_3) -> /Arduino Connector/SPI5_MOSI
- CN2 pad 4: Net-(CN2-Pin_4) -> /Arduino Connector/SPI5_MISO
- CN2 pad 5: Net-(CN2-Pin_5) -> /Arduino Connector/SPI5_CLK
- CN2 pad 6: Net-(CN2-Pin_6) -> CPU_C-DIR
- CN3 pad 1: unconnected-(CN3-Pin_1-Pad1) -> CPU_B-STEP
- CN3 pad 10: Net-(CN3-Pin_10) -> /Arduino Connector/I2C_SCL
- CN3 pad 2: Net-(CN3-Pin_2) -> CPU_A-STEP
- CN3 pad 3: unconnected-(CN3-Pin_3-Pad3) -> SPINDLESPEED
- CN3 pad 4: Net-(CN3-Pin_4) -> /Arduino Connector/PWM12_2
- CN3 pad 5: unconnected-(CN3-Pin_5-Pad5) -> /Arduino Connector/PWM12_1
- CN3 pad 6: Net-(CN3-Pin_6) -> INPUT_INT
- CN3 pad 9: Net-(CN3-Pin_9) -> /Arduino Connector/I2C_SDA
- CN4 pad 1: Net-(CN4-Pin_1) -> /Arduino Connector/PWM8_2
- CN4 pad 2: Net-(CN4-Pin_2) -> CPU_X-STEP
- CN4 pad 3: Net-(CN4-Pin_3) -> CPU_Y-STEP
- CN4 pad 4: Net-(CN4-Pin_4) -> CPU_Z-STEP
- CN4 pad 5: Net-(CN4-Pin_5) -> CPU_X-DIR
- CN4 pad 6: Net-(CN4-Pin_6) -> CPU_Y-DIR
- CN4 pad 7: Net-(CN4-Pin_7) -> CPU_Z-DIR
- CN4 pad 8: Net-(CN4-Pin_8) -> CPU_C-STEP

Commit message: wip Kicad
Parts:
- removed PS1: B0503LS-1WR3, stm32F746 GRBL:CONV_B0503LS-1WR3
- removed Q1, Q2, Q3: STD30NF06, Package_TO_SOT_SMD:TO-252-2
- added C4: 100nF, Capacitor_SMD:C_0805_2012Metric, B.Cu at (108.8, 82.0)
- added RJ1: 0R, stm32F746 GRBL:RJ_3 pads_0805_2012Metric, B.Cu at (117.5, 73.8)
- added RJ10: 0R, stm32F746 GRBL:RJ_3 pads_0805_2012Metric, B.Cu at (152.2, 73.8)
- added RJ11: 0R, stm32F746 GRBL:RJ_3 pads_0805_2012Metric, B.Cu at (165.2, 73.8)
- added RJ12: 0R, stm32F746 GRBL:RJ_3 pads_0805_2012Metric, B.Cu at (167.5, 73.8)
- added RJ13: 0R, stm32F746 GRBL:RJ_3 pads_0805_2012Metric, B.Cu at (169.8, 73.8)
- added RJ14: 0R, stm32F746 GRBL:RJ_3 pads_0805_2012Metric, B.Cu at (172.0, 73.8)
- added RJ15: 0R, stm32F746 GRBL:RJ_3 pads_0805_2012Metric, B.Cu at (174.2, 73.8)
- added RJ16: 0R, stm32F746 GRBL:RJ_3 pads_0805_2012Metric, B.Cu at (117.5, 98.8)
- added RJ17: 0R, stm32F746 GRBL:RJ_3 pads_0805_2012Metric, B.Cu at (119.8, 98.8)
- added RJ18: 0R, stm32F746 GRBL:RJ_3 pads_0805_2012Metric, B.Cu at (122.0, 98.8)
- added RJ19: 0R, stm32F746 GRBL:RJ_3 pads_0805_2012Metric, B.Cu at (124.2, 98.8)
- added RJ2: 0R, stm32F746 GRBL:RJ_3 pads_0805_2012Metric, B.Cu at (119.8, 73.8)
- added RJ20: 0R, stm32F746 GRBL:RJ_3 pads_0805_2012Metric, B.Cu at (126.5, 98.8)
- added RJ21: 0R, stm32F746 GRBL:RJ_3 pads_0805_2012Metric, B.Cu at (143.2, 98.8)
- added RJ22: 0R, stm32F746 GRBL:RJ_3 pads_0805_2012Metric, B.Cu at (145.5, 98.8)
- added RJ23: 0R, stm32F746 GRBL:RJ_3 pads_0805_2012Metric, B.Cu at (147.8, 98.8)
- added RJ24: 0R, stm32F746 GRBL:RJ_3 pads_0805_2012Metric, B.Cu at (150.0, 98.8)
- added RJ25: 0R, stm32F746 GRBL:RJ_3 pads_0805_2012Metric, B.Cu at (152.2, 98.8)
- added RJ26: 0R, stm32F746 GRBL:RJ_3 pads_0805_2012Metric, B.Cu at (165.5, 98.7)
- added RJ27: 0R, stm32F746 GRBL:RJ_3 pads_0805_2012Metric, B.Cu at (167.8, 98.7)
- added RJ28: 0R, stm32F746 GRBL:RJ_3 pads_0805_2012Metric, B.Cu at (170.0, 98.7)
- added RJ29: 0R, stm32F746 GRBL:RJ_3 pads_0805_2012Metric, B.Cu at (172.2, 98.7)
- added RJ3: 0R, stm32F746 GRBL:RJ_3 pads_0805_2012Metric, B.Cu at (122.0, 73.8)
- added RJ30: 0R, stm32F746 GRBL:RJ_3 pads_0805_2012Metric, B.Cu at (174.5, 98.7)
- added RJ4: 0R, stm32F746 GRBL:RJ_3 pads_0805_2012Metric, B.Cu at (124.2, 73.8)
- added RJ5: 0R, stm32F746 GRBL:RJ_3 pads_0805_2012Metric, B.Cu at (126.5, 73.8)
- added RJ6: 0R, stm32F746 GRBL:RJ_3 pads_0805_2012Metric, B.Cu at (143.2, 73.8)
- added RJ7: 0R, stm32F746 GRBL:RJ_3 pads_0805_2012Metric, B.Cu at (145.5, 73.8)
- added RJ8: 0R, stm32F746 GRBL:RJ_3 pads_0805_2012Metric, B.Cu at (147.8, 73.8)
- added RJ9: 0R, stm32F746 GRBL:RJ_3 pads_0805_2012Metric, B.Cu at (150.0, 73.8)
- added RN1: 4K7, Resistor_THT:R_Array_SIP9, F.Cu at (101.5, 70.8)
- added RN2: 4K7, Resistor_THT:R_Array_SIP9, F.Cu at (101.5, 94.7)
- added U7: TLP521-4, Package_SO:SOIC-16_4.55x10.3mm_P1.27mm, F.Cu at (94.8, 98.2)
- added U8: TLP521-4, Package_SO:SOIC-16_4.55x10.3mm_P1.27mm, F.Cu at (94.8, 109.8)
- C3, U3: moved to B.Cu
- J14: value Screw_Terminal_01x09 -> Input 1-8
- J15: value Screw_Terminal_01x09 -> Input 9-16
- J16: value Screw_Terminal_01x09 -> Output
- U4: value XTR115U -> MCP23017_SS; footprint Package_SO:SOIC-8_3.9x4.9mm_P1.27mm -> Package_SO:SSOP-28_5.3x10.2mm_P0.65mm; moved to B.Cu
- moved U3 42.3 mm to (133.2, 111.5)
- moved C3 36.3 mm to (133.2, 115.8)
- moved U9 32.4 mm to (169.8, 87.0), turned to 90 degrees
- moved U4 31.7 mm to (109.9, 75.7), turned to 90 degrees
- moved D7 29.6 mm to (166.0, 87.0)
- moved R13 26.4 mm to (169.5, 90.0), turned to 0 degrees
- moved C1 24.5 mm to (110.5, 84.5)
- moved C2 17.1 mm to (110.0, 110.8), turned to 90 degrees
- moved U1 5.68 mm to (110.0, 77.2)
- moved J16 3.68 mm to (112.8, 64.2)
- moved U6 3.58 mm to (94.8, 86.8)
- moved U5 3.56 mm to (94.8, 75.2)
- moved U2 3.36 mm to (110.0, 102.2)
- moved J14 2.06 mm to (83.5, 93.9)
- moved J15 2.06 mm to (83.5, 69.4)
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- renumbered U7 to U9
Connections:
- net INPUT_1 renamed /Input/INPUT_1
- net INPUT_2 renamed /Input/INPUT_2
- net INPUT_3 renamed /Input/INPUT_3
- net INPUT_4 renamed /Input/INPUT_4
- net INPUT_5 renamed /Input/INPUT_5
- net INPUT_6 renamed /Input/INPUT_6
- net INPUT_7 renamed /Input/INPUT_7
- net INPUT_8 renamed /Input/INPUT_8
- A1 pad 10: unconnected-(A1-CFG0-Pad10) -> Net-(A1-CFG0)
- A1 pad 11: unconnected-(A1-CFG1-Pad11) -> Net-(A1-CFG1)
- A1 pad 12: unconnected-(A1-CFG2-Pad12) -> Net-(A1-CFG2)
- A1 pad 13: unconnected-(A1-CFG3-Pad13) -> Net-(A1-CFG3)
- A1 pad 14: unconnected-(A1-CFG4-Pad14) -> Net-(A1-CFG4)
- A2 pad 10: unconnected-(A2-CFG0-Pad10) -> Net-(A2-CFG0)
- A2 pad 11: unconnected-(A2-CFG1-Pad11) -> Net-(A2-CFG1)
- A2 pad 12: unconnected-(A2-CFG2-Pad12) -> Net-(A2-CFG2)
- A2 pad 13: unconnected-(A2-CFG3-Pad13) -> Net-(A2-CFG3)
- A2 pad 14: unconnected-(A2-CFG4-Pad14) -> Net-(A2-CFG4)
- A2 pad 15: /Driver/Z-STEP -> /Driver/Y-STEP
- A2 pad 16: /Driver/Z-DIR -> /Driver/Y-DIR
- A3 pad 10: unconnected-(A3-CFG0-Pad10) -> Net-(A3-CFG0)
- A3 pad 11: unconnected-(A3-CFG1-Pad11) -> Net-(A3-CFG1)
- A3 pad 12: unconnected-(A3-CFG2-Pad12) -> Net-(A3-CFG2)
- A3 pad 13: unconnected-(A3-CFG3-Pad13) -> Net-(A3-CFG3)
- A3 pad 14: unconnected-(A3-CFG4-Pad14) -> Net-(A3-CFG4)
- A3 pad 15: /Driver/Y-STEP -> /Driver/Z-STEP
- A3 pad 16: /Driver/Y-DIR -> /Driver/Z-DIR
- A4 pad 10: unconnected-(A4-CFG0-Pad10) -> Net-(A4-CFG0)
- A4 pad 11: unconnected-(A4-CFG1-Pad11) -> Net-(A4-CFG1)
- A4 pad 12: unconnected-(A4-CFG2-Pad12) -> Net-(A4-CFG2)
- A4 pad 13: unconnected-(A4-CFG3-Pad13) -> Net-(A4-CFG3)
- A4 pad 14: unconnected-(A4-CFG4-Pad14) -> Net-(A4-CFG4)
- A5 pad 10: unconnected-(A5-CFG0-Pad10) -> Net-(A5-CFG0)
- A5 pad 11: unconnected-(A5-CFG1-Pad11) -> Net-(A5-CFG1)
- A5 pad 12: unconnected-(A5-CFG2-Pad12) -> Net-(A5-CFG2)
- A5 pad 13: unconnected-(A5-CFG3-Pad13) -> Net-(A5-CFG3)
- A5 pad 14: unconnected-(A5-CFG4-Pad14) -> Net-(A5-CFG4)
- A6 pad 10: unconnected-(A6-CFG0-Pad10) -> Net-(A6-CFG0)
- A6 pad 11: unconnected-(A6-CFG1-Pad11) -> Net-(A6-CFG1)
- A6 pad 12: unconnected-(A6-CFG2-Pad12) -> Net-(A6-CFG2)
- A6 pad 13: unconnected-(A6-CFG3-Pad13) -> Net-(A6-CFG3)
- A6 pad 14: unconnected-(A6-CFG4-Pad14) -> Net-(A6-CFG4)
- C1 pad 1: +3.3V -> +3.3VP
- C2 pad 1: +3.3V -> +3.3VP
- CN1 pad 3: /Arduino Connector/RESET -> RESET
- CN2 pad 1: CPU_A-DIR -> unconnected-(CN2-Pin_1-Pad1)
- CN2 pad 2: CPU_B-DIR -> unconnected-(CN2-Pin_2-Pad2)
- CN2 pad 3: /Arduino Connector/SPI5_MOSI -> CPU_C-DIR
- CN2 pad 4: /Arduino Connector/SPI5_MISO -> CPU_C-STEP
- CN2 pad 5: /Arduino Connector/SPI5_CLK -> CPU_Z-DIR
- CN2 pad 6: CPU_C-DIR -> CPU_Z-STEP
- CN3 pad 1: CPU_B-STEP -> CPU_B-DIR
- CN3 pad 10: /Arduino Connector/I2C_SCL -> I2C_SCL
- CN3 pad 2: CPU_A-STEP -> CPU_ENABLE
- CN3 pad 5: /Arduino Connector/PWM12_1 -> INPUT_INT_1
- CN3 pad 6: INPUT_INT -> INPUT_INT_2
- CN3 pad 9: /Arduino Connector/I2C_SDA -> I2C_SDA
- CN4 pad 3: CPU_Y-STEP -> CPU_X-DIR
- CN4 pad 4: CPU_Z-STEP -> CPU_Y-STEP
- CN4 pad 5: CPU_X-DIR -> CPU_Y-DIR
- CN4 pad 6: CPU_Y-DIR -> CPU_A-STEP
- CN4 pad 7: CPU_Z-DIR -> CPU_A-DIR
- CN4 pad 8: CPU_C-STEP -> CPU_B-STEP
- D7 pad 3: CPU_X-STEP -> CPU_ENABLE
- J14 pad 1: unconnected-(J14-Pin_1-Pad1) -> GND
- J15 pad 1: unconnected-(J15-Pin_1-Pad1) -> GND
- J16 pad 9: unconnected-(J16-Pin_9-Pad9) -> GND
- R13 pad 1: CPU_X-STEP -> CPU_ENABLE
- U1 pad 1: /IO_Expansion/I2C_SCL -> I2C_SCL
- U1 pad 18: +3.3V -> +3.3VP
- U1 pad 2: /IO_Expansion/I2C_SDA -> I2C_SDA
- U1 pad 6: /IO_Expansion/RESET -> RESET
- U1 pad 8: /IO_Expansion/INPUT_INT -> INPUT_INT_1
- U2 pad 1: /IO_Expansion/I2C_SCL -> I2C_SCL
- U2 pad 10: INPUT_9 -> /Input/INPUT_9
- U2 pad 11: INPUT_10 -> /Input/INPUT_10
- U2 pad 12: INPUT_11 -> /Input/INPUT_11
- U2 pad 13: INPUT_12 -> /Input/INPUT_12
- U2 pad 14: INPUT_13 -> /Input/INPUT_13
- U2 pad 15: INPUT_14 -> /Input/INPUT_14
- U2 pad 16: INPUT_15 -> /Input/INPUT_15
- U2 pad 17: INPUT_16 -> /Input/INPUT_16
- U2 pad 18: +3.3V -> +3.3VP
- U2 pad 2: /IO_Expansion/I2C_SDA -> I2C_SDA
- U2 pad 5: +3.3V -> +3.3VP
- U2 pad 6: /IO_Expansion/RESET -> RESET
- U2 pad 8: /IO_Expansion/INPUT_INT -> INPUT_INT_2
- U3 pad 5: /Arduino Connector/I2C_SDA -> I2C_SDA
- U3 pad 6: /Arduino Connector/I2C_SCL -> I2C_SCL
- U5 pad 2: GNDPWR -> unconnected-(U5-Pad2)
- U5 pad 4: GNDPWR -> unconnected-(U5-Pad4)
- U5 pad 6: GNDPWR -> unconnected-(U5-Pad6)
- U5 pad 8: GNDPWR -> unconnected-(U5-Pad8)
- U6 pad 2: GNDPWR -> unconnected-(U6-Pad2)
- U6 pad 4: GNDPWR -> unconnected-(U6-Pad4)
- U6 pad 6: GNDPWR -> unconnected-(U6-Pad6)
- U6 pad 8: GNDPWR -> unconnected-(U6-Pad8)
- U9 pad 1: unconnected-(U7-Pad1) -> +3.3VP
- U9 pad 5: unconnected-(U7-VCC-Pad5) -> +3.3VP
Other:
- board text added: "A"
- board text added: "AXIS-A"
- board text added: "AXIS-B"
- board text added: "AXIS-C"
- board text added: "AXIS-X"
- board text added: "AXIS-Y"
- board text added: "AXIS-Z"
- board text added: "B"
- board text added: "C"
- board text added: "X"
- board text added: "Y"
- board text added: "Z"
