File: Kicad/stm32F746 GRBL/stm32F746 GRBL.kicad_pcb (KiCad board)
At the start: 2 copper layers, 130 x 80 mm, 95 parts, among them CN1 PinHeader_1x08_P2.54mm_Vertic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, CN2 PinHeader_1x06_P2.54mm_Vertic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, CN3 PinHeader_1x10_P2.54mm_Vertic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, CN4 PinHeader_1x08_P2.54mm_Vertic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, J1 X-Axis, J10 Conn_01x04, J11 Conn_01x04, J12 Conn_01x04, J13 Screw_Terminal_01x04, J14 Input 1-8, J15 Input 9-16, J16 Output, J2 Y-Axis, J3 Z-Axis, J4 A-Axis, J5 B-Axis, J6 C-Axis, J7 Conn_01x04, J8 Conn_01x04, J9 Conn_01x04, U1 MCP23008-xSO, U2 MCP23008-xSO, U3 24LC64, U4 MCP23017_SS, U5 TLP521-4, U6 TLP521-4, U7 TLP521-4, U8 TLP521-4, U9 74AHCT1G125

Commit message: kicad wip
Parts:
- added C5: 2.2uF, Capacitor_SMD:C_0805_2012Metric_Pad1.18x1.45mm_HandSolder, F.Cu at (156.2, 121.0)
- added C6: 0.1uF, Capacitor_SMD:C_0805_2012Metric, F.Cu at (158.1, 114.0)
- added C7: 22uF, Capacitor_SMD:C_0805_2012Metric_Pad1.18x1.45mm_HandSolder, F.Cu at (149.8, 113.5)
- added C8: 22uF, Capacitor_SMD:C_0805_2012Metric_Pad1.18x1.45mm_HandSolder, F.Cu at (149.7, 111.0)
- added C9: 10uF, Capacitor_Tantalum_SMD:CP_EIA-3528-15_AVX-H_Pad1.50x2.35mm_HandSolder, F.Cu at (153.1, 127.9)
- added F1: Polyfuse, Fuse:Fuse_1812_4532Metric_Pad1.30x3.40mm_HandSolder, F.Cu at (159.8, 125.2)
- added J17: PWM-1, Connector_PinHeader_2.54mm:PinHeader_1x03_P2.54mm_Vertical, F.Cu at (84.2, 65.6)
- added J18: PWM-2, Connector_PinHeader_2.54mm:PinHeader_1x03_P2.54mm_Vertical, F.Cu at (88.0, 65.6)
- added J19: PWM-3, Connector_PinHeader_2.54mm:PinHeader_1x03_P2.54mm_Vertical, F.Cu at (91.8, 65.6)
- added J20: PWM-4, Connector_PinHeader_2.54mm:PinHeader_1x03_P2.54mm_Vertical, F.Cu at (95.5, 65.6)
- added L1: 6.8uH, Inductor_SMD:L_Bourns_SRP5030T, F.Cu at (151.0, 117.8)
- added Q1: BSS138, Package_TO_SOT_SMD:SOT-23, F.Cu at (100.1, 65.8)
- added Q2: BSS138, Package_TO_SOT_SMD:SOT-23, F.Cu at (107.3, 65.8)
- added Q3: BSS138, Package_TO_SOT_SMD:SOT-23, B.Cu at (107.3, 65.8)
- added Q4: BSS138, Package_TO_SOT_SMD:SOT-23, B.Cu at (100.1, 65.8)
- added R14: 100K, Resistor_SMD:R_0805_2012Metric_Pad1.20x1.40mm_HandSolder, F.Cu at (162.5, 117.8)
- added R15: 13.7K, Resistor_SMD:R_0805_2012Metric_Pad1.20x1.40mm_HandSolder, F.Cu at (160.2, 117.8)
- added R16: 10K, Resistor_SMD:R_0805_2012Metric_Pad1.20x1.40mm_HandSolder, F.Cu at (103.2, 65.8)
- added R17: 10K, Resistor_SMD:R_0805_2012Metric_Pad1.20x1.40mm_HandSolder, F.Cu at (99.1, 62.0)
- added R18: 10K, Resistor_SMD:R_0805_2012Metric_Pad1.20x1.40mm_HandSolder, F.Cu at (110.4, 65.8)
- added R19: 10K, Resistor_SMD:R_0805_2012Metric_Pad1.20x1.40mm_HandSolder, F.Cu at (106.4, 62.0)
- added R20: 10K, Resistor_SMD:R_0805_2012Metric_Pad1.20x1.40mm_HandSolder, B.Cu at (110.4, 65.8)
- added R21: 10K, Resistor_SMD:R_0805_2012Metric_Pad1.20x1.40mm_HandSolder, B.Cu at (106.4, 62.0)
- added R22: 10K, Resistor_SMD:R_0805_2012Metric_Pad1.20x1.40mm_HandSolder, B.Cu at (103.2, 65.8)
- added R23: 10K, Resistor_SMD:R_0805_2012Metric_Pad1.20x1.40mm_HandSolder, B.Cu at (99.1, 62.0)
- added RN3: 390, Package_SO:SOIC-16_4.55x10.3mm_P1.27mm, B.Cu at (89.8, 79.5)
- added RN4: 390, Package_SO:SOIC-16_4.55x10.3mm_P1.27mm, B.Cu at (89.8, 104.3)
- added RN5: 4K7, Resistor_THT:R_Array_SIP9, F.Cu at (95.5, 70.9)
- added RN6: 4K7, Resistor_THT:R_Array_SIP9, F.Cu at (95.5, 95.3)
- added U10: LMR51430, Package_TO_SOT_SMD:SOT-23-6, F.Cu at (157.0, 117.8)
- added U11: LM1117MP-3.3, Package_TO_SOT_SMD:SOT-223-3_TabPin2, F.Cu at (146.6, 127.2)
- added U12: ULN2803A, Package_SO:SOIC-18W_7.5x11.6mm_P1.27mm, B.Cu at (125.8, 114.8)
- C1, C2: moved to B.Cu
- C3, C4, U3, U4: moved to F.Cu
- J13: value Screw_Terminal_01x04 -> Power Input
- J14: renamed from J15; value Input 9-16 -> Input 1-8
- J15: renamed from J14; value Input 1-8 -> Input 9-16
- J16: footprint TerminalBlock_TE-Connectivity:TerminalBlock_TE_282834-9_1x09_P2.54mm_Horizontal -> TerminalBlock_TE-Connectivity:TerminalBlock_TE_1-282834-0_1x10_P2.54mm_Horizontal
- U1, U2: value MCP23008-xSO -> MCP23008-xSS; footprint Package_SO:SOIC-18W_7.5x11.6mm_P1.27mm -> Package_SO:SSOP-20_5.3x7.2mm_P0.65mm; moved to B.Cu
- moved J13 76.5 mm to (168.6, 120.7)
- moved J1 75.8 mm to (200.2, 71.0), turned to 180 degrees
- moved J16 67.5 mm to (88.4, 127.2), turned to 0 degrees
- moved J2 62.8 mm to (200.2, 81.5), turned to 180 degrees
- moved J3 49.8 mm to (200.2, 92.0), turned to 180 degrees
- moved C4 43.1 mm to (127.0, 121.0)
- moved U4 41.2 mm to (124.2, 114.2), turned to 180 degrees
- moved J4 37.0 mm to (200.2, 102.5), turned to 180 degrees
- moved J5 24.6 mm to (200.2, 113.0), turned to 180 degrees
- moved J6 13.5 mm to (200.0, 123.5), turned to 180 degrees
- moved U1 11.2 mm to (113.0, 88.0), turned to -90 degrees
- moved U2 11.2 mm to (113.0, 113.0), turned to -90 degrees
- moved C2 8.52 mm to (118.2, 113.0), turned to -90 degrees
- moved C1 8.46 mm to (118.2, 88.0), turned to 90 degrees
- moved U7 7.13 mm to (101.5, 100.5)
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Connections:
- CN2 pad 1: unconnected-(CN2-Pin_1-Pad1) -> PWM3
- CN2 pad 2: unconnected-(CN2-Pin_2-Pad2) -> CPU_C-DIR
- CN2 pad 3: CPU_C-DIR -> PWM4
- CN3 pad 4: /Arduino Connector/PWM12_2 -> PWM1
- CN4 pad 1: /Arduino Connector/PWM8_2 -> PWM2
- J13 pad 2: unconnected-(J13-Pin_2-Pad2) -> Vdrive
- J13 pad 3: unconnected-(J13-Pin_3-Pad3) -> GND
- J14 pad 1: GND -> /Input/IN1
- J14 pad 2: unconnected-(J15-Pin_2-Pad2) -> /Input/IN2
- J14 pad 3: unconnected-(J15-Pin_3-Pad3) -> /Input/IN3
- J14 pad 4: unconnected-(J15-Pin_4-Pad4) -> /Input/IN4
- J14 pad 5: unconnected-(J15-Pin_5-Pad5) -> /Input/IN5
- J14 pad 6: unconnected-(J15-Pin_6-Pad6) -> /Input/IN6
- J14 pad 7: unconnected-(J15-Pin_7-Pad7) -> /Input/IN7
- J14 pad 8: unconnected-(J15-Pin_8-Pad8) -> /Input/IN8
- J14 pad 9: unconnected-(J15-Pin_9-Pad9) -> GND
- J15 pad 1: GND -> /Input/IN9
- J15 pad 2: unconnected-(J14-Pin_2-Pad2) -> /Input/IN10
- J15 pad 3: unconnected-(J14-Pin_3-Pad3) -> /Input/IN11
- J15 pad 4: unconnected-(J14-Pin_4-Pad4) -> /Input/IN12
- J15 pad 5: unconnected-(J14-Pin_5-Pad5) -> /Input/IN13
- J15 pad 6: unconnected-(J14-Pin_6-Pad6) -> /Input/IN14
- J15 pad 7: unconnected-(J14-Pin_7-Pad7) -> /Input/IN15
- J15 pad 8: unconnected-(J14-Pin_8-Pad8) -> /Input/IN16
- J15 pad 9: unconnected-(J14-Pin_9-Pad9) -> GND
- J16 pad 1: unconnected-(J16-Pin_1-Pad1) -> Net-(J16-Pin_1)
- J16 pad 2: unconnected-(J16-Pin_2-Pad2) -> Net-(J16-Pin_2)
- J16 pad 3: unconnected-(J16-Pin_3-Pad3) -> Net-(J16-Pin_3)
- J16 pad 4: unconnected-(J16-Pin_4-Pad4) -> Net-(J16-Pin_4)
- J16 pad 5: unconnected-(J16-Pin_5-Pad5) -> Net-(J16-Pin_5)
- J16 pad 6: unconnected-(J16-Pin_6-Pad6) -> Net-(J16-Pin_6)
- J16 pad 7: unconnected-(J16-Pin_7-Pad7) -> Net-(J16-Pin_7)
- J16 pad 8: unconnected-(J16-Pin_8-Pad8) -> Net-(J16-Pin_8)
- J16 pad 9: GND -> Net-(J16-Pin_9)
- U1 pad 10: /Input/INPUT_1 -> unconnected-(U1-NC-Pad10)
- U1 pad 11: /Input/INPUT_2 -> unconnected-(U1-NC-Pad11)
- U1 pad 12: /Input/INPUT_3 -> /Input/INPUT_1
- U1 pad 13: /Input/INPUT_4 -> /Input/INPUT_2
- U1 pad 14: /Input/INPUT_5 -> /Input/INPUT_3
- U1 pad 15: /Input/INPUT_6 -> /Input/INPUT_4
- U1 pad 16: /Input/INPUT_7 -> /Input/INPUT_5
- U1 pad 17: /Input/INPUT_8 -> /Input/INPUT_6
- U1 pad 18: +3.3VP -> /Input/INPUT_7
- U2 pad 10: /Input/INPUT_9 -> unconnected-(U2-NC-Pad10)
- U2 pad 11: /Input/INPUT_10 -> unconnected-(U2-NC-Pad11)
- U2 pad 12: /Input/INPUT_11 -> /Input/INPUT_9
- U2 pad 13: /Input/INPUT_12 -> /Input/INPUT_10
- U2 pad 14: /Input/INPUT_13 -> /Input/INPUT_11
- U2 pad 15: /Input/INPUT_14 -> /Input/INPUT_12
- U2 pad 16: /Input/INPUT_15 -> /Input/INPUT_13
- U2 pad 17: /Input/INPUT_16 -> /Input/INPUT_14
- U2 pad 18: +3.3VP -> /Input/INPUT_15
- U4 pad 1: unconnected-(U4-GPB0-Pad1) -> Net-(U12-I1)
- U4 pad 2: unconnected-(U4-GPB1-Pad2) -> Net-(U12-I2)
- U4 pad 21: unconnected-(U4-GPA0-Pad21) -> /Output/SPINDLE_ENABLE
- U4 pad 3: unconnected-(U4-GPB2-Pad3) -> Net-(U12-I3)
- U4 pad 4: unconnected-(U4-GPB3-Pad4) -> Net-(U12-I4)
- U4 pad 5: unconnected-(U4-GPB4-Pad5) -> Net-(U12-I5)
- U4 pad 6: unconnected-(U4-GPB5-Pad6) -> Net-(U12-I6)
- U4 pad 7: unconnected-(U4-GPB6-Pad7) -> Net-(U12-I7)
- U4 pad 8: unconnected-(U4-GPB7-Pad8) -> Net-(U12-I8)
- U5 pad 1: unconnected-(U5-Pad1) -> Net-(RN3A-R1.1)
- U5 pad 2: unconnected-(U5-Pad2) -> GND
- U5 pad 3: unconnected-(U5-Pad3) -> Net-(RN3B-R2.1)
- U5 pad 4: unconnected-(U5-Pad4) -> GND
- U5 pad 5: unconnected-(U5-Pad5) -> Net-(RN3C-R3.1)
- U5 pad 6: unconnected-(U5-Pad6) -> GND
- U5 pad 7: unconnected-(U5-Pad7) -> Net-(RN3D-R4.1)
- U5 pad 8: unconnected-(U5-Pad8) -> GND
- U6 pad 1: unconnected-(U6-Pad1) -> Net-(RN3E-R5.1)
- U6 pad 2: unconnected-(U6-Pad2) -> GND
- U6 pad 3: unconnected-(U6-Pad3) -> Net-(RN3F-R6.1)
- U6 pad 4: unconnected-(U6-Pad4) -> GND
- U6 pad 5: unconnected-(U6-Pad5) -> Net-(RN3G-R7.1)
- U6 pad 6: unconnected-(U6-Pad6) -> GND
- U6 pad 7: unconnected-(U6-Pad7) -> Net-(RN3H-R8.1)
- U6 pad 8: unconnected-(U6-Pad8) -> GND
- U7 pad 1: unconnected-(U7-Pad1) -> Net-(RN4A-R1.1)
- U7 pad 2: unconnected-(U7-Pad2) -> GND
- U7 pad 3: unconnected-(U7-Pad3) -> Net-(RN4B-R2.1)
- U7 pad 4: unconnected-(U7-Pad4) -> GND
- U7 pad 5: unconnected-(U7-Pad5) -> Net-(RN4C-R3.1)
- U7 pad 6: unconnected-(U7-Pad6) -> GND
- U7 pad 7: unconnected-(U7-Pad7) -> Net-(RN4D-R4.1)
- U7 pad 8: unconnected-(U7-Pad8) -> GND
- U8 pad 1: unconnected-(U8-Pad1) -> Net-(RN4E-R5.1)
- U8 pad 2: unconnected-(U8-Pad2) -> GND
- U8 pad 3: unconnected-(U8-Pad3) -> Net-(RN4F-R6.1)
- U8 pad 4: unconnected-(U8-Pad4) -> GND
- U8 pad 5: unconnected-(U8-Pad5) -> Net-(RN4G-R7.1)
- U8 pad 6: unconnected-(U8-Pad6) -> GND
- U8 pad 7: unconnected-(U8-Pad7) -> Net-(RN4H-R8.1)
- U8 pad 8: unconnected-(U8-Pad8) -> GND
Routing:
- net /Driver/ENABLE: track 0.00 -> 42.0 mm
- net Net-(A6-2B): track 0.00 -> 6.08 mm
- net Net-(A6-2A): track 0.00 -> 6.06 mm
- net Net-(A5-1B): track 0.00 -> 6.05 mm
- net Net-(A4-1B): track 0.00 -> 6.05 mm
- net Net-(A3-1B): track 0.00 -> 6.05 mm
- net Net-(A2-1B): track 0.00 -> 6.05 mm
- net Net-(A1-1B): track 0.00 -> 6.05 mm
- net Net-(A6-1A): track 0.00 -> 6.05 mm
- net Net-(A5-1A): track 0.00 -> 6.03 mm
- net Net-(A3-1A): track 0.00 -> 6.03 mm
- net Net-(A2-1A): track 0.00 -> 6.03 mm
- net Net-(A4-1A): track 0.00 -> 6.03 mm
- net Net-(A1-1A): track 0.00 -> 6.03 mm
- net Net-(A6-1B): track 0.00 -> 6.03 mm
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Other:
- board text added: "IN-1"

Commit message: wip kicad
Parts:
- added C10: 10nF, Capacitor_SMD:C_0805_2012Metric, F.Cu at (127.2, 141.4)
- added C11: 10nF, Capacitor_SMD:C_0805_2012Metric, F.Cu at (127.2, 144.4)
- added C12: 0.1uF, Capacitor_SMD:C_0805_2012Metric, F.Cu at (127.2, 147.4)
- added C14: 470nF, Capacitor_SMD:C_0805_2012Metric, F.Cu at (127.2, 150.4)
- added D9: SMAJ40CA, Diode_SMD:D_SMA, F.Cu at (113.0, 123.5)
- added J21: 4-20MA or 0-10V, TerminalBlock_TE-Connectivity:TerminalBlock_TE_282834-2_1x02_P2.54mm_Horizontal, F.Cu at (111.6, 129.5)
- added Q5: MMBT5087, Package_TO_SOT_SMD:SOT-23, F.Cu at (137.1, 155.0)
- added Q6: BSP170, Package_TO_SOT_SMD:SOT-223-3_TabPin2, F.Cu at (134.4, 144.0)
- added R24: 4K7, Resistor_SMD:R_0805_2012Metric_Pad1.20x1.40mm_HandSolder, F.Cu at (122.6, 141.3)
- added R25: 8K25, Resistor_SMD:R_0805_2012Metric_Pad1.20x1.40mm_HandSolder, F.Cu at (122.6, 144.3)
- added R26: 5K62, Resistor_SMD:R_0805_2012Metric_Pad1.20x1.40mm_HandSolder, F.Cu at (122.6, 147.2)
- added R27: 1K65, Resistor_SMD:R_0805_2012Metric_Pad1.20x1.40mm_HandSolder, F.Cu at (122.6, 150.2)
- added R28: 15, Resistor_SMD:R_0805_2012Metric_Pad1.20x1.40mm_HandSolder, F.Cu at (122.6, 153.2)
- added R29: 15, Resistor_SMD:R_0805_2012Metric_Pad1.20x1.40mm_HandSolder, F.Cu at (122.6, 156.1)
- added R30: 10K, Resistor_SMD:R_0805_2012Metric_Pad1.20x1.40mm_HandSolder, F.Cu at (122.6, 159.1)
- added U13: XTR111AxDGQ, Package_SO:MSOP-10-1EP_3x3mm_P0.5mm_EP2.2x3.1mm_Mask1.83x1.89mm_ThermalVias, F.Cu at (133.1, 150.4)
- added U14: TSV911RILT, Package_TO_SOT_SMD:SOT-23-5, F.Cu at (132.0, 155.0)
- moved U12 37.9 mm to (88.5, 121.5), turned to -90 degrees
- moved C4 10.2 mm to (120.5, 113.2), turned to -90 degrees
- moved U4 10.1 mm to (114.2, 113.8)
- moved J16 4.34 mm to (84.7, 129.5)
- moved J13 4.25 mm to (168.6, 125.0)
- moved J14 2.51 mm to (81.0, 70.9)
- moved J15 2.51 mm to (81.0, 95.4)
- moved RN3 0.25 mm to (89.5, 79.5)
- moved RN4 0.25 mm to (89.5, 104.3)
Connections:
- C5 pad 1: Net-(U10-EN) -> Vdrive
- F1 pad 1: Vdrive -> Net-(J13-Pin_1)
- F1 pad 2: Net-(U10-EN) -> Vdrive
- J13 pad 1: Vdrive -> Net-(J13-Pin_1)
- J13 pad 2: Vdrive -> Net-(J13-Pin_1)
- U10 pad 3: Net-(U10-EN) -> Vdrive
- U10 pad 5: Net-(U10-EN) -> Vdrive
- U4 pad 1: Net-(U12-I1) -> Net-(U12-I8)
- U4 pad 2: Net-(U12-I2) -> Net-(U12-I7)
- U4 pad 27: unconnected-(U4-GPA6-Pad27) -> /Output/ERROR_FLAG
- U4 pad 28: unconnected-(U4-GPA7-Pad28) -> /Output/4_20MA_OR_0_10V_DISABLE
- U4 pad 3: Net-(U12-I3) -> Net-(U12-I6)
- U4 pad 4: Net-(U12-I4) -> Net-(U12-I5)
- U4 pad 5: Net-(U12-I5) -> Net-(U12-I4)
- U4 pad 6: Net-(U12-I6) -> Net-(U12-I3)
- U4 pad 7: Net-(U12-I7) -> Net-(U12-I2)
- U4 pad 8: Net-(U12-I8) -> Net-(U12-I1)
Other:
- board text added: "1"
- board text added: "10"
- board text added: "11"
- board text added: "12"
- board text added: "13"
- board text added: "14"
- board text added: "15"
- board text added: "16"
- board text added: "2"
- board text added: "3"
- board text added: "4"
- board text added: "5"
- board text added: "6"
- board text added: "7"
- board text added: "8"
- board text added: "9"
- board text added: "GND"
- board text added: "INPUT"
- board text added: "OUTPUT"
- board text added: "POWER"
- board text added: "V+"
- board text removed: "IN-1"

Commit message: kicad wip
Parts:
- added C13: 4.7uF, Capacitor_SMD:C_0805_2012Metric, F.Cu at (93.0, 158.8)
- added D8: SS16-E3, Diode_SMD:D_SMA, F.Cu at (154.5, 163.8)
- C5, C6, C7, C8, C9, L1, R14, R15, U10, U11: moved to B.Cu
- moved C12 39.6 mm to (89.2, 158.6), turned to -90 degrees
- moved U14 38.9 mm to (94.2, 164.1), turned to -90 degrees
- moved R24 38.7 mm to (91.2, 163.9), turned to -90 degrees
- moved C11 34.8 mm to (160.5, 134.0)
- moved F1 32.5 mm to (191.8, 131.0), turned to 90 degrees
- moved C8 25.3 mm to (172.7, 121.5)
- moved C5 24.9 mm to (179.2, 111.5)
- moved R27 24.0 mm to (145.2, 142.2), turned to -90 degrees
- moved C7 23.6 mm to (172.8, 119.0)
- moved C6 23.4 mm to (181.1, 118.5), turned to -90 degrees
- moved Q6 23.3 mm to (154.8, 132.8), turned to 90 degrees
- moved L1 23.2 mm to (174.0, 114.8)
- moved R14 23.2 mm to (185.5, 114.8), turned to 90 degrees
- moved R15 23.2 mm to (183.2, 114.8), turned to -90 degrees
- moved U10 23.2 mm to (180.0, 114.8)
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Connections:
- U13 pad 1: unconnected-(U13-VSP-Pad1) -> Vdrive
