File: Kicad/stm32F746 GRBL/Output.kicad_sch (KiCad schematic)
At the start: 3 parts, among them Q1 STD30NF06, Q2 STD30NF06, Q3 STD30NF06

Commit message: wip kicad
Parts:
- added J16: Screw_Terminal_01x09, TerminalBlock_TE-Connectivity:TerminalBlock_TE_282834-9_1x09_P2.54mm_Horizontal, symbol Connector:Screw_Terminal_01x09
- added U4: XTR115U, Package_SO:SOIC-8_3.9x4.9mm_P1.27mm, symbol Interface_CurrentLoop:XTR115U
Changed lines of the file:
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@@
 (kicad_sch (version 20230121) (generator eeschema)
   (paper "A4")
-  (label "SPINDLE_SPEED" (at 215.9 107.95 180) (fields_autoplaced)
+  (label "SPINDLE_SPEED" (at 205.74 38.1 180) (fields_autoplaced)
     (effects (font (size 1.27 1.27)) (justify right bottom))
   )
+  (symbol (lib_id "Connector:Screw_Terminal_01x09") (at 72.39 72.39 180) (unit 1)
+    (in_bom yes) (on_board yes) (dnp no) (fields_autoplaced)
+    (property "Reference" "J16" (at 72.39 55.88 0)
+      (effects (font (size 1.27 1.27)))
+    )
+    (property "Value" "Screw_Terminal_01x09" (at 72.39 58.42 0)
+      (effects (font (size 1.27 1.27)))
+    )
+    (property "Footprint" "TerminalBlock_TE-Connectivity:TerminalBlock_TE_282834-9_1x09_P2.54mm_Horizontal" (at 72.39 72.39 0)
+      (effects (font (size 1.27 1.27)) hide)
+    )
+    (property "Datasheet" "~" (at 72.39 72.39 0)
+      (effects (font (size 1.27 1.27)) hide)
+    )
+    (pin "6")
+    (pin "1")
+    (pin "4")
+    (pin "7")
+    (pin "2")
+    (pin "8")
+    (pin "5")
+    (pin "3")
+    (pin "9")
+    (instances
+      (project "stm32F746 GRBL"
+        (path "/2c79a78e-687a-4954-b7b9-175bc3470bd7/eddc17cf-fbda-41ce-9eec-af5043ce77b7"
+          (reference "J16") (unit 1)
+        )
+      )
+    )
+  )
+  (symbol (lib_id "Interface_CurrentLoop:XTR115U") (at 138.43 92.71 0) (unit 1)
+    (in_bom yes) (on_board yes) (dnp no) (fields_autoplaced)
+    (property "Reference" "U4" (at 138.43 74.93 0)
+      (effects (font (size 1.27 1.27)))
+    )
+    (property "Value" "XTR115U" (at 138.43 77.47 0)
+      (effects (font (size 1.27 1.27)))
+    )
+    (property "Footprint" "Package_SO:SOIC-8_3.9x4.9mm_P1.27mm" (at 138.43 102.87 0)
+      (effects (font (size 1.27 1.27)) hide)
+    )
+    (property "Datasheet" "http://www.ti.com/lit/ds/symlink/xtr115.pdf" (at 138.43 92.71 0)
+      (effects (font (size 1.27 1.27)) hide)
+    )
+    (pin "2")
+    (pin "6")
+    (pin "8")
+    (pin "4")
+    (pin "5")
+    (pin "7")
+    (pin "3")
+    (pin "1")
+    (instances
+      (project "stm32F746 GRBL"
+        (path "/2c79a78e-687a-4954-b7b9-175bc3470bd7/eddc17cf-fbda-41ce-9eec-af5043ce77b7"
+          (reference "U4") (unit 1)
+        )
+      )
+    )
+  )
   (symbol (lib_id "STD30nf06:STD30NF06") (at 227.33 58.42 0) (unit 1)

Commit message: wip Kicad
Parts:
- removed Q1, Q2, Q3: STD30NF06, Package_TO_SOT_SMD:TO-252-2, symbol STD30nf06:STD30NF06
- removed U4: XTR115U, Package_SO:SOIC-8_3.9x4.9mm_P1.27mm, symbol Interface_CurrentLoop:XTR115U
- added C4: 100nF, Capacitor_SMD:C_0805_2012Metric, symbol Device:C
- added U4: MCP23017_SS, Package_SO:SSOP-28_5.3x10.2mm_P0.65mm, symbol Interface_Expansion:MCP23017_SS
- J16: value Screw_Terminal_01x09 -> Output
Connections:
- net GND: now reaches J16.9 (Pin_9)
- net GND: now also C4.2, U4.10 (VSS), U4.15 (A0), U4.16 (A1)
- new net +3.3VP: C4.1, U4.17 (A2), U4.9 (VDD)
- new net I2C_SCL: U4.12 (SCK)
- new net I2C_SDA: U4.13 (SDA)
- new net RESET: U4.18 (~{RESET})
- no-connect marks 0 -> 2
Other:
- note added: "0x24 - 0100(100)x"
- moved on the sheet: J16

Commit message: kicad wip
Parts:
- removed J16: Output, TerminalBlock_TE-Connectivity:TerminalBlock_TE_282834-9_1x09_P2.54mm_Horizontal, symbol Connector:Screw_Terminal_01x09
- added J16: Output, TerminalBlock_TE-Connectivity:TerminalBlock_TE_1-282834-0_1x10_P2.54mm_Horizontal, symbol Connector:Screw_Terminal_01x10
- added J17: PWM-1, Connector_PinHeader_2.54mm:PinHeader_1x03_P2.54mm_Vertical, symbol Connector_Generic:Conn_01x03
- added J18: PWM-2, Connector_PinHeader_2.54mm:PinHeader_1x03_P2.54mm_Vertical, symbol Connector_Generic:Conn_01x03
- added J19: PWM-3, Connector_PinHeader_2.54mm:PinHeader_1x03_P2.54mm_Vertical, symbol Connector_Generic:Conn_01x03
- added J20: PWM-4, Connector_PinHeader_2.54mm:PinHeader_1x03_P2.54mm_Vertical, symbol Connector_Generic:Conn_01x03
- added Q1, Q2, Q3, Q4: BSS138, Package_TO_SOT_SMD:SOT-23, symbol Transistor_FET:BSS138
- added R16, R17, R18, R19, R20, R21, R22, R23, R24: 10K, Resistor_SMD:R_0805_2012Metric_Pad1.20x1.40mm_HandSolder, symbol Device:R
- added U12: ULN2803A, Package_SO:SOIC-18W_7.5x11.6mm_P1.27mm, symbol Transistor_Array:ULN2803A
- added U13: TS921, Package_SO:TSSOP-8_4.4x3mm_P0.65mm, symbol stm32F746 GRBL:TS921
- added U14: TLP185, Package_SO:SOIC-4_4.55x3.7mm_P2.54mm, symbol Isolator:TLP185
Connections:
- net +3.3VP: now also Q1.1 (G), Q2.1 (G), Q3.1 (G), Q4.1 (G), R16.1, R18.1, R20.1, R22.1
- net GND: now also J16.10 (Pin_10), J17.3 (Pin_3), J18.3 (Pin_3), J19.3 (Pin_3), J20.3 (Pin_3), U12.9 (GND), U13.4 (V-), U14.3
- net at U4.1 (GPB0): now also U12.1 (I1)
- net at U4.2 (GPB1): now also U12.2 (I2)
- net SPINDLE_ENABLE: now reaches U4.21 (GPA0)
- net at U4.3 (GPB2): now also U12.3 (I3)
- net at U4.4 (GPB3): now also U12.4 (I4)
- net at U4.5 (GPB4): now also U12.5 (I5)
- net at U4.6 (GPB5): now also U12.6 (I6)
- net at U4.7 (GPB6): now also U12.7 (I7)
- net at U4.8 (GPB7): now also U12.8 (I8)
- new net: J17.1 (Pin_1), Q1.3 (D), R17.2
- new net: J19.1 (Pin_1), Q3.3 (D), R21.2
- new net: J16.1 (Pin_1), U12.10 (COM)
- new net: J16.9 (Pin_9), U12.11 (O8)
- new net: J16.8 (Pin_8), U12.12 (O7)
- new net: J16.7 (Pin_7), U12.13 (O6)
- new net: J16.6 (Pin_6), U12.14 (O5)
- new net: J16.5 (Pin_5), U12.15 (O4)
- new net: J16.4 (Pin_4), U12.16 (O3)
- new net: J16.3 (Pin_3), U12.17 (O2)
- new net: J16.2 (Pin_2), U12.18 (O1)
- new net: J20.1 (Pin_1), Q4.3 (D), R23.2
- new net: R24.2, U14.1
- new net: J18.1 (Pin_1), Q2.3 (D), R19.2
- new net +5VP: J17.2 (Pin_2), J18.2 (Pin_2), J19.2 (Pin_2), J20.2 (Pin_2), R17.1, R19.1, R21.1, R23.1
- new net PWM1: Q1.2 (S), R16.2
- new net PWM2: Q2.2 (S), R18.2
- new net PWM3: Q3.2 (S), R20.2
- new net PWM4: Q4.2 (S), R22.2
- new net SPINDLESPEED: R24.1
Other:
- note added: "EXT_V+_REF"

Commit message: wip kicad
Parts:
- removed U13: TS921, Package_SO:TSSOP-8_4.4x3mm_P0.65mm, symbol stm32F746 GRBL:TS921
- removed U14: TLP185, Package_SO:SOIC-4_4.55x3.7mm_P2.54mm, symbol Isolator:TLP185
- added C10, C11: 10nF, Capacitor_SMD:C_0805_2012Metric, symbol Device:C
- added C12: 0.1uF, Capacitor_SMD:C_0805_2012Metric, symbol Device:C
- added C13: 4.7uF, Capacitor_SMD:C_0805_2012Metric, symbol Device:C_Polarized
- added C14: 470nF, Capacitor_SMD:C_0805_2012Metric, symbol Device:C
- added D8: SS16-E3, symbol Device:D_Schottky
- added D9: SMAJ40CA, Diode_SMD:D_SMA, symbol Diode:SMAJ40CA
- added J21: 4-20MA or 0-10V, TerminalBlock_TE-Connectivity:TerminalBlock_TE_282834-2_1x02_P2.54mm_Horizontal, symbol Connector:Screw_Terminal_01x02
- added Q5: MMBT5087, Package_TO_SOT_SMD:SOT-23, symbol Transistor_BJT:MMBT3906
- added Q6: BSP170, Package_TO_SOT_SMD:SOT-223-3_TabPin2, symbol Transistor_FET:ZXMP4A16G
- added R25: 8K25, Resistor_SMD:R_0805_2012Metric_Pad1.20x1.40mm_HandSolder, symbol Device:R
- added R26: 5K62, Resistor_SMD:R_0805_2012Metric_Pad1.20x1.40mm_HandSolder, symbol Device:R
- added R27: 1K65, Resistor_SMD:R_0805_2012Metric_Pad1.20x1.40mm_HandSolder, symbol Device:R
- added R28, R29: 15, Resistor_SMD:R_0805_2012Metric_Pad1.20x1.40mm_HandSolder, symbol Device:R
- added R30: 10K, Resistor_SMD:R_0805_2012Metric_Pad1.20x1.40mm_HandSolder, symbol Device:R
- added U13: XTR111AxDGQ, Package_SO:MSOP-10-1EP_3x3mm_P0.5mm_EP2.2x3.1mm_Mask1.83x1.89mm_ThermalVias, symbol Interface_CurrentLoop:XTR111AxDGQ
- added U14: TSV911RILT, Package_TO_SOT_SMD:SOT-23-5, symbol Amplifier_Operational:TSV911RILT
- R24: value 10K -> 4K7
Connections:
- net +3.3VP: now also R30.2
- net GND: now also C10.2, C11.2, C12.2, C13.2, C14.1, D9.1 (A1), J21.2 (Pin_2), R25.2, R27.1, U13.10 (GND), U13.11 (GND), U14.5 (V-)
- net at U4.1 (GPB0): now also U12.8 (I8); no longer U12.1 (I1)
- net at U4.2 (GPB1): now also U12.7 (I7); no longer U12.2 (I2)
- net at U4.3 (GPB2): now also U12.6 (I6); no longer U12.3 (I3)
- net at U4.4 (GPB3): now also U12.5 (I5); no longer U12.4 (I4)
- net at U4.5 (GPB4): now also U12.4 (I4); no longer U12.5 (I5)
- net at U4.6 (GPB5): now also U12.3 (I3); no longer U12.6 (I6)
- net at U4.7 (GPB6): now also U12.2 (I2); no longer U12.7 (I7)
- net at U4.8 (GPB7): now also U12.1 (I1); no longer U12.8 (I8)
- net at R24.2: now also C13.1, U14.3 (+)
- net ERROR_FLAG: now reaches U4.27 (GPA6)
- net ERROR_FLAG: now also R30.1, U13.8 (~{EF})
- net 4_20MA_OR_0_10V_DISABLE: now reaches U4.28 (GPA7)
- net 4_20MA_OR_0_10V_DISABLE: now also U13.9 (OD)
- new net: Q5.3 (C), Q6.1 (G), U13.3 (VG)
- new net: Q5.1 (B), Q6.2 (D), R28.2
- new net: C11.1, D8.1 (K), Q6.3 (S), R29.1
- new net: R25.1, R26.2, U13.4 (REGS)
- new net: U13.6 (VIN), U14.1, U14.4 (-)
- new net: Q5.2 (E), R28.1, U13.2 (IS)
- new net: R27.2, U13.7 (SET)
- new net: D9.2 (A2), J21.1 (Pin_1), R29.2
- new net +5VD: C12.1, C14.2, R26.1, U13.5 (REGF), U14.2 (V+)
- new net Vdrive: C10.1, D8.2 (A)
Other:
- note added: "IOUT = 10x(VIN/RSET)"
- moved on the sheet: C4, J17, J18, J19, J20, Q1, Q2, Q3, Q4, R16, R17, R18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

Commit message: kicad wip
Parts:
- D8: footprint (none) -> Diode_SMD:D_SMA; Digikey (none) -> SS16-E3/61TGICT-ND
Connections:
- net Vdrive: now also U13.1 (VSP)
Other:
- moved on the sheet: J21
Changed lines of the file:
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@@
   (junction (at 66.675 128.27) (diameter 0) (color 0 0 0 0)
   )
-  (junction (at 100.965 107.95) (diameter 0) (color 0 0 0 0)
-  )
   (junction (at 172.72 150.495) (diameter 0) (color 0 0 0 0)
   )
   (junction (at 88.9 111.125) (diameter 0) (color 0 0 0 0)
+  )
+  (junction (at 100.965 111.125) (diameter 0) (color 0 0 0 0)
   )
   (junction (at 55.88 78.105) (diameter 0) (color 0 0 0 0)
@@
     (stroke (width 0) (type default))
   )
-  (wire (pts (xy 100.965 107.315) (xy 100.965 107.95))
-    (stroke (width 0) (type default))
-  )
   (wire (pts (xy 57.15 78.105) (xy 55.88 78.105))
     (stroke (width 0) (type default))
@@
     (stroke (width 0) (type default))
   )
-  (wire (pts (xy 172.72 150.495) (xy 206.375 150.495))
+  (wire (pts (xy 172.72 150.495) (xy 189.865 150.495))
     (stroke (width 0) (type default))
   )
@@
     (stroke (width 0) (type default))
   )
-  (wire (pts (xy 100.965 107.95) (xy 100.965 111.125))
+  (wire (pts (xy 100.965 107.315) (xy 100.965 111.125))
     (stroke (width 0) (type default))
   )
@@
     (stroke (width 0) (type default))
   )
-  (wire (pts (xy 205.74 153.035) (xy 206.375 153.035))
+  (wire (pts (xy 189.23 153.035) (xy 189.865 153.035))
     (stroke (width 0) (type default))
   )
@@
     (stroke (width 0) (type default))
   )
-  (wire (pts (xy 205.74 153.035) (xy 205.74 154.94))
+  (wire (pts (xy 189.23 153.035) (xy 189.23 154.94))
     (stroke (width 0) (type default))
   )
@@
     (stroke (width 0) (type default))
   )
-  (wire (pts (xy 100.965 111.76) (xy 100.965 115.57))
+  (wire (pts (xy 100.965 111.125) (xy 100.965 115.57))
     (stroke (width 0) (type default))
   )
@@
       (effects (font (size 1.27 1.27)) (justify right))
     )
-    (property "Footprint" "" (at 154.94 144.145 0)
-      (effects (font (size 1.27 1.27)) hide)
-    )
-    (property "Datasheet" "~" (at 154.94 144.145 0)
+    (property "Footprint" "Diode_SMD:D_SMA" (at 154.94 144.145 0)
+      (effects (font (size 1.27 1.27)) hide)
+    )
+    (property "Datasheet" "https://www.vishay.com/docs/88746/ss12.pdf" (at 154.94 144.145 0)
+      (effects (font (size 1.27 1.27)) hide)
+    )
+    (property "Digikey" "SS16-E3/61TGICT-ND" (at 154.94 144.145 90)
       (effects (font (size 1.27 1.27)) hide)
     )
@@
     )
   )
-  (symbol (lib_id "power:Vdrive") (at 100.965 107.95 0) (unit 1)
-    (in_bom yes) (on_board yes) (dnp no)
-    (property "Reference" "#PWR011" (at 95.885 111.76 0)
-      (effects (font (size 1.27 1.27)) hide)
-    )
-    (property "Value" "Vdrive" (at 106.045 105.41 0)
-      (effects (font (size 1.27 1.27)))
-    )
-    (property "Footprint" "" (at 100.965 107.95 0)
-      (effects (font (size 1.27 1.27)) hide)
-    )
-    (property "Datasheet" "" (at 100.965 107.95 0)
+  (symbol (lib_id "power:Vdrive") (at 100.965 107.315 0) (unit 1)
+    (in_bom yes) (on_board yes) (dnp no)
+    (property "Reference" "#PWR011" (at 95.885 111.125 0)
+      (effects (font (size 1.27 1.27)) hide)
+    )
+    (property "Value" "Vdrive" (at 106.045 104.775 0)
+      (effects (font (size 1.27 1.27)))
+    )
+    (property "Footprint" "" (at 100.965 107.315 0)
+      (effects (font (size 1.27 1.27)) hide)
+    )
+    (property "Datasheet" "" (at 100.965 107.315 0)
       (effects (font (size 1.27 1.27)) hide)
     )
@@
     )
   )
-  (symbol (lib_id "power:GND") (at 205.74 154.94 0) (unit 1)
-    (in_bom yes) (on_board yes) (dnp no)
-    (property "Reference" "#PWR096" (at 205.74 161.29 0)
-      (effects (font (size 1.27 1.27)) hide)
-    )
-    (property "Value" "GND" (at 201.93 158.75 0)
-      (effects (font (size 1.27 1.27)) hide)
-    )
-    (property "Footprint" "" (at 205.74 154.94 0)
-      (effects (font (size 1.27 1.27)) hide)
-    )
-    (property "Datasheet" "" (at 205.74 154.94 0)
+  (symbol (lib_id "power:GND") (at 189.23 154.94 0) (unit 1)
+    (in_bom yes) (on_board yes) (dnp no)
+    (property "Reference" "#PWR096" (at 189.23 161.29 0)
+      (effects (font (size 1.27 1.27)) hide)
+    )
+    (property "Value" "GND" (at 185.42 158.75 0)
+      (effects (font (size 1.27 1.27)) hide)
+    )
+    (property "Footprint" "" (at 189.23 154.94 0)
+      (effects (font (size 1.27 1.27)) hide)
+    )
+    (property "Datasheet" "" (at 189.23 154.94 0)
       (effects (font (size 1.27 1.27)) hide)
     )
@@
     )
   )
-  (symbol (lib_id "Connector:Screw_Terminal_01x02") (at 211.455 150.495 0) (unit 1)
-    (in_bom yes) (on_board yes) (dnp no)
-    (property "Reference" "J21" (at 210.185 147.32 0)
-      (effects (font (size 1.27 1.27)) (justify left))
-    )
-    (property "Value" "4-20MA or 0-10V" (at 213.995 151.765 0)
-      (effects (font (size 1.27 1.27)) (justify left))
-    )
-    (property "Footprint" "TerminalBlock_TE-Connectivity:TerminalBlock_TE_282834-2_1x02_P2.54mm_Horizontal" (at 211.455 150.495 0)
-      (effects (font (size 1.27 1.27)) hide)
-    )
-    (property "Datasheet" "~" (at 211.455 150.495 0)
-      (effects (font (size 1.27 1.27)) hide)
-    )
+  (symbol (lib_id "Connector:Screw_Terminal_01x02") (at 194.945 150.495 0) (unit 1)
+    (in_bom yes) (on_board yes) (dnp no)
+    (property "Reference" "J21" (at 193.675 147.32 0)
+      (effects (font (size 1.27 1.27)) (justify left))
+    )
+    (property "Value" "4-20MA or 0-10V" (at 197.485 151.765 0)
+      (effects (font (size 1.27 1.27)) (justify left))
+    )
+    (property "Footprint" "TerminalBlock_TE-Connectivity:TerminalBlock_TE_282834-2_1x02_P2.54mm_Horizontal" (at 194.945 150.495 0)
+      (effects (font (size 1.27 1.27)) hide)
+    )
+    (property "Datasheet" "~" (at 194.945 150.495 0)
+      (effects (font (size 1.27 1.27)) hide)
+    )

Commit message: wip kicad
Connections:
- net SPINDLESPEED renamed PWM_4-20MA
- no-connect marks 2 -> 7
Changed lines of the file:
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@@
   )
   (no_connect (at 57.15 55.245))
+  (no_connect (at 92.71 73.025))
   (no_connect (at 57.15 52.705))
+  (no_connect (at 92.71 62.865))
+  (no_connect (at 92.71 70.485))
+  (no_connect (at 92.71 65.405))
+  (no_connect (at 92.71 67.945))
   (wire (pts (xy 231.775 121.285) (xy 231.775 121.92))
     (stroke (width 0) (type default))
@@
     )
   )
-  (global_label "SPINDLESPEED" (shape input) (at 34.29 125.73 180) (fields_autoplaced)
+  (global_label "PWM_4-20MA" (shape input) (at 34.29 125.73 180) (fields_autoplaced)
     (effects (font (size 1.27 1.27)) (justify right))
-    (property "Intersheetrefs" "${INTERSHEET_REFS}" (at 17.3954 125.73 0)
+    (property "Intersheetrefs" "${INTERSHEET_REFS}" (at 18.4235 125.73 0)
       (effects (font (size 1.27 1.27)) (justify right) hide)
     )
