File: Kicad/stm32F746 GRBL/Driver.kicad_sch (KiCad schematic)
At the start: 18 parts, among them J1 X-Axis, J10 Conn_01x04, J11 Conn_01x04, J12 Conn_01x04, J2 Y-Axis, J3 Z-Axis, J4 A-Axis, J5 B-Axis, J6 C-Axis, J7 Conn_01x04, J8 Conn_01x04, J9 Conn_01x04

Commit message: wip
Parts:
- added D1, D2, D3, D4, D5, D6: 2BZX84C3V9, Package_TO_SOT_SMD:SOT-23, symbol Diode:2BZX84Cxx
- added D7: BZX84Cxx, Package_TO_SOT_SMD:SOT-23, symbol Diode:BZX84Cxx
- added R1, R10, R11, R12, R13, R2, R3, R4, R5, R6, R7, R8, R9: 270, Resistor_SMD:R_0805_2012Metric, symbol Device:R
- added U7: 74AHCT1G125, Package_TO_SOT_SMD:SOT-353_SC-70-5, symbol 74xGxx:74AHCT1G125
Connections:
- net A-DIR: now also R8.2
- net A-STEP: now also R7.2
- net B-DIR: now also R10.2
- net B-STEP: now also R9.2
- net C-DIR: now also R12.2
- net C-STEP: now also R11.2
- net ENABLE: now also U7.4
- net GND: now also D1.3 (A), D2.3 (A), D3.3 (A), D4.3 (A), D5.3 (A), D6.3 (A), D7.1 (A), U7.3 (GND)
- net X-DIR: now also R2.2
- net X-STEP: now also R1.2
- net Y-DIR: now also R4.2
- net Y-STEP: now also R3.2
- net Z-DIR: now also R6.2
- net Z-STEP: now also R5.2
- new net: R13.2, U7.2
- new net CPU_A-DIR: D4.1 (K), R8.1
- new net CPU_A-STEP: D4.2 (K), R7.1
- new net CPU_B-DIR: D5.1 (K), R10.1
- new net CPU_B-STEP: D5.2 (K), R9.1
- new net CPU_C-DIR: D6.1 (K), R12.1
- new net CPU_C-STEP: D6.2 (K), R11.1
- new net CPU_X-DIR: D1.1 (K), R2.1
- new net CPU_X-STEP: D1.2 (K), D7.3 (K), R1.1, R13.1
- new net CPU_Y-DIR: D2.1 (K), R4.1
- new net CPU_Y-STEP: D2.2 (K), R3.1
- new net CPU_Z-DIR: D3.1 (K), R6.1
- new net CPU_Z-STEP: D3.2 (K), R5.1
Other:
- moved on the sheet: A1, A2, A3, A4, A5, A6, J1, J10, J11, J12, J2, J3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

Commit message: wip Kicad
Parts:
- added RJ1, RJ10, RJ11, RJ12, RJ13, RJ14, RJ15, RJ16, RJ17, RJ18, RJ19, RJ2, RJ20, RJ21, RJ22, RJ23, RJ24, RJ25, RJ26, RJ27, RJ28, RJ29, RJ3, RJ30, RJ4, RJ5, RJ6, RJ7, RJ8, RJ9: 0R, stm32F746 GRBL:RJ_3 pads_0805_2012Metric, symbol stm32F746 GRBL:RJ
- renumbered U7 to U9
Connections:
- net CPU_X-STEP: no longer D7.3 (K), R13.1
- net GND: now also RJ1.3, RJ10.3, RJ11.3, RJ12.3, RJ13.3, RJ14.3, RJ15.3, RJ16.3, RJ17.3, RJ18.3, RJ19.3, RJ2.3, RJ20.3, RJ21.3, RJ22.3, RJ23.3, RJ24.3, RJ25.3, RJ26.3, RJ27.3, RJ28.3, RJ29.3, RJ3.3, RJ30.3, RJ4.3, RJ5.3, RJ6.3, RJ7.3, RJ8.3, RJ9.3
- net Y-DIR: now also A2.16 (DIR); no longer A3.16 (DIR)
- net Y-STEP: now also A2.15 (STEP); no longer A3.15 (STEP)
- net Z-DIR: now also A3.16 (DIR); no longer A2.16 (DIR)
- net Z-STEP: now also A3.15 (STEP); no longer A2.15 (STEP)
- net at A4.10 (CFG0): now also RJ16.2
- net at A4.11 (CFG1): now also RJ17.2
- net at A4.12 (CFG2): now also RJ18.2
- net at A4.13 (CFG3): now also RJ19.2
- net at A4.14 (CFG4): now also RJ20.2
- net at A5.10 (CFG0): now also RJ21.2
- net at A5.11 (CFG1): now also RJ22.2
- net at A5.12 (CFG2): now also RJ23.2
- net at A5.13 (CFG3): now also RJ24.2
- net at A5.14 (CFG4): now also RJ25.2
- net at A6.10 (CFG0): now also RJ26.2
- net at A6.11 (CFG1): now also RJ27.2
- net at A6.12 (CFG2): now also RJ28.2
- net at A6.13 (CFG3): now also RJ29.2
- net at A6.14 (CFG4): now also RJ30.2
- net at A1.10 (CFG0): now also RJ1.2
- net at A1.11 (CFG1): now also RJ2.2
- net at A1.12 (CFG2): now also RJ3.2
- net at A1.13 (CFG3): now also RJ5.2
- net at A1.14 (CFG4): now also RJ4.2
- net +3.3VP: now reaches U9.1
- net +3.3VP: now also U9.5 (VCC), RJ1.1, RJ10.1, RJ11.1, RJ12.1, RJ13.1, RJ14.1, RJ15.1, RJ16.1, RJ17.1, RJ18.1, RJ19.1, RJ2.1, RJ20.1, RJ21.1, RJ22.1, RJ23.1, RJ24.1, RJ25.1, RJ26.1, RJ27.1, RJ28.1, RJ29.1, RJ3.1, RJ30.1, RJ4.1, RJ5.1, RJ6.1, RJ7.1, RJ8.1, RJ9.1
- net at A3.10 (CFG0): now also RJ11.2
- net at A3.11 (CFG1): now also RJ12.2
- net at A3.12 (CFG2): now also RJ13.2
- net at A3.13 (CFG3): now also RJ14.2
- net at A3.14 (CFG4): now also RJ15.2
- net at A2.10 (CFG0): now also RJ6.2
- net at A2.11 (CFG1): now also RJ7.2
- net at A2.12 (CFG2): now also RJ8.2
- net at A2.13 (CFG3): now also RJ9.2
- net at A2.14 (CFG4): now also RJ10.2
- new net CPU_ENABLE: D7.3 (K), R13.1
Other:
- moved on the sheet: A1, A2, A3, A4, A5, A6, D1, D2, D3, D4, D5, D6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

Commit message: wip Kicad.
Parts:
- renumbered RJ5 to RJ4, RJ4 to RJ5
Changed lines of the file:
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@@
   (symbol (lib_id "stm32F746 GRBL:RJ") (at 23.495 44.45 0) (unit 1)
     (in_bom yes) (on_board yes) (dnp no)
-    (property "Reference" "RJ5" (at 23.495 39.37 90)
+    (property "Reference" "RJ4" (at 23.495 39.37 90)
       (effects (font (size 1.27 1.27)) (justify right))
     )
@@
       (project "stm32F746 GRBL"
         (path "/2c79a78e-687a-4954-b7b9-175bc3470bd7/8d1e1584-2808-4a74-84c8-15e2fc5b3024"
-          (reference "RJ5") (unit 1)
+          (reference "RJ4") (unit 1)
         )
       )
@@
   (symbol (lib_id "stm32F746 GRBL:RJ") (at 19.685 44.45 0) (unit 1)
     (in_bom yes) (on_board yes) (dnp no)
-    (property "Reference" "RJ4" (at 19.685 39.37 90)
+    (property "Reference" "RJ5" (at 19.685 39.37 90)
       (effects (font (size 1.27 1.27)) (justify right))
     )
@@
       (project "stm32F746 GRBL"
         (path "/2c79a78e-687a-4954-b7b9-175bc3470bd7/8d1e1584-2808-4a74-84c8-15e2fc5b3024"
-          (reference "RJ4") (unit 1)
-        )
-      )
+          (reference "RJ5") (unit 1)
+        )
+      )
